File: hardware/radartof-hardware.kicad_pcb (KiCad board)
At the start: 2 copper layers, 66 x 66 mm, 22 parts, among them J1 Debug, J2 J3026G01DNLT, U1 ABX00042, U2 VL53L5CXV0GC/1

Commit message: final-ish schematic
Parts:
- added C10: 100n, Capacitor_SMD:C_0603_1608Metric, F.Cu at (231.7, 108.4)
- added C11: 100n, Capacitor_SMD:C_0603_1608Metric, F.Cu at (235.7, 100.9)
- added C12: 10u, Capacitor_SMD:C_0603_1608Metric, F.Cu at (235.7, 103.4)
- added C13: 10u, Capacitor_SMD:C_0603_1608Metric, F.Cu at (235.7, 105.9)
- added C14: 10u, Capacitor_SMD:C_0603_1608Metric, F.Cu at (235.7, 108.4)
- added C15: 10u, Capacitor_SMD:C_0603_1608Metric, F.Cu at (239.8, 100.9)
- added C16: 1n, Capacitor_SMD:C_0603_1608Metric, F.Cu at (222.4, 74.9)
- added C17: 10n, Capacitor_SMD:C_0402_1005Metric, F.Cu at (201.4, 100.9)
- added C18: 10u, Capacitor_SMD:C_0603_1608Metric, F.Cu at (201.4, 103.4)
- added C19: 10u, Capacitor_SMD:C_0603_1608Metric, F.Cu at (201.4, 105.9)
- added C20: 10u, Capacitor_SMD:C_0603_1608Metric, F.Cu at (201.4, 108.4)
- added C21: 1u, Capacitor_SMD:C_0603_1608Metric, F.Cu at (201.4, 110.9)
- added C22: 10n, Capacitor_SMD:C_0402_1005Metric, F.Cu at (201.4, 113.5)
- added C23: 100n, Capacitor_SMD:C_0603_1608Metric, F.Cu at (201.4, 116.0)
- added C24: 10u, Capacitor_SMD:C_0603_1608Metric, F.Cu at (201.4, 118.5)
- added C25: 10n, Capacitor_SMD:C_0402_1005Metric, F.Cu at (205.4, 100.9)
- added C26: 10u, Capacitor_SMD:C_0603_1608Metric, F.Cu at (205.4, 103.4)
- added C27: 10u, Capacitor_SMD:C_0603_1608Metric, F.Cu at (205.4, 105.9)
- added C28: 10n, Capacitor_SMD:C_0402_1005Metric, F.Cu at (205.4, 108.4)
- added C29: 10u, Capacitor_SMD:C_0603_1608Metric, F.Cu at (205.4, 110.9)
- added C30: 1u, Capacitor_SMD:C_0603_1608Metric, F.Cu at (205.4, 113.5)
- added C31: 10n, Capacitor_SMD:C_0402_1005Metric, F.Cu at (205.4, 116.0)
- added C32: 1u, Capacitor_SMD:C_0603_1608Metric, F.Cu at (205.4, 118.5)
- added C33: 1u, Capacitor_SMD:C_0603_1608Metric, F.Cu at (209.4, 100.9)
- added C34: 10n, Capacitor_SMD:C_0402_1005Metric, F.Cu at (209.4, 103.4)
- added C35: 10n, Capacitor_SMD:C_0402_1005Metric, F.Cu at (209.4, 105.9)
- added C36: 1u, Capacitor_SMD:C_0603_1608Metric, F.Cu at (209.4, 108.4)
- added C37: 10n, Capacitor_SMD:C_0402_1005Metric, F.Cu at (209.4, 110.9)
- added C38: 1u, Capacitor_SMD:C_0603_1608Metric, F.Cu at (209.4, 113.5)
- added C39: 10n, Capacitor_SMD:C_0402_1005Metric, F.Cu at (209.4, 116.0)
- added C40: 1u, Capacitor_SMD:C_0603_1608Metric, F.Cu at (209.4, 118.5)
- added C41: 10n, Capacitor_SMD:C_0402_1005Metric, F.Cu at (213.4, 100.9)
- added C42: 470n, Capacitor_SMD:C_0603_1608Metric, F.Cu at (213.4, 103.4)
- added C43: 1u, Capacitor_SMD:C_0603_1608Metric, F.Cu at (213.4, 105.9)
- added C44: 100n, Capacitor_SMD:C_0603_1608Metric, F.Cu at (206.2, 81.5)
- added C45: 100n, Capacitor_SMD:C_0603_1608Metric, F.Cu at (206.2, 84.0)
- added C46: 100n, Capacitor_SMD:C_0603_1608Metric, F.Cu at (206.2, 86.5)
- added C7: 100n, Capacitor_SMD:C_0603_1608Metric, F.Cu at (231.7, 100.9)
- added C8: 100n, Capacitor_SMD:C_0603_1608Metric, F.Cu at (231.7, 103.4)
- added C9: 100n, Capacitor_SMD:C_0603_1608Metric, F.Cu at (231.7, 105.9)
- added FB1: FerriteBead, Capacitor_SMD:C_0603_1608Metric, F.Cu at (239.8, 103.4)
- added J3: Camera, OV5640:OV2640FSL, F.Cu at (166.5, 115.0)
- added J4: J3026G01DNLT, J3026G01DNLT:PE_J3026G01DNLT, F.Cu at (175.0, 72.0)
- added JP1: VIO Select, Jumper:SolderJumper-3_P1.3mm_Open_RoundedPad1.0x1.5mm, F.Cu at (237.7, 116.0)
- added L1: L, Inductor_SMD:L_0603_1608Metric, F.Cu at (200.9, 130.7)
- added L2: L, Inductor_SMD:L_0603_1608Metric, F.Cu at (200.9, 133.2)
- added L3: L, Inductor_SMD:L_0603_1608Metric, F.Cu at (200.9, 135.7)
- added L4: L, Inductor_SMD:L_0603_1608Metric, F.Cu at (200.9, 138.2)
- added L5: L, Inductor_SMD:L_0603_1608Metric, F.Cu at (200.9, 140.8)
- added L6: L, Inductor_SMD:L_0603_1608Metric, F.Cu at (200.9, 143.3)
- added L7: L, Inductor_SMD:L_0603_1608Metric, F.Cu at (200.9, 145.8)
- added R13: 10k, Resistor_SMD:R_0603_1608Metric, F.Cu at (239.8, 105.9)
- added R14: 10k, Resistor_SMD:R_0603_1608Metric, F.Cu at (239.8, 108.4)
- added R15: 5k1, Resistor_SMD:R_0603_1608Metric, F.Cu at (230.5, 72.4)
- added R16: 5k1, Resistor_SMD:R_0603_1608Metric, F.Cu at (230.5, 74.9)
- added R17: 1M, Resistor_SMD:R_0603_1608Metric, F.Cu at (230.5, 77.4)
- added R18: 150, Resistor_SMD:R_0603_1608Metric, F.Cu at (213.4, 108.4)
- added TP1: Vmotor, TestPoint:TestPoint_Pad_D1.5mm, F.Cu at (227.9, 101.4)
- added TP2: GNDmotor, TestPoint:TestPoint_Pad_D1.5mm, F.Cu at (227.9, 105.0)
- added TP3: Strobe, TestPoint:TestPoint_Pad_D1.5mm, F.Cu at (227.9, 108.5)
- added U10: KC2016Z24.0000, Oscillator:Oscillator_SMD_Kyocera_KC2520Z-4Pin_2.5x2.0mm, F.Cu at (236.9, 112.0)
- added U11: USBLC6-2SC6, Package_TO_SOT_SMD:SOT-23-6, F.Cu at (201.6, 82.5)
- added U12: USBLC6-2SC6, Package_TO_SOT_SMD:SOT-23-6, F.Cu at (201.6, 86.9)
- added U13: USBLC6-2SC6, Package_TO_SOT_SMD:SOT-23-6, F.Cu at (137.0, 90.0)
- added U3: TLV74328 SOT23-5, Package_TO_SOT_SMD:SOT-23-5, F.Cu at (232.3, 111.9)
- added U4: TLV74315 SOT23-5, Package_TO_SOT_SMD:SOT-23-5, F.Cu at (232.3, 116.4)
- added U5: TLV74318 SOT23-5, Package_TO_SOT_SMD:SOT-23-5, F.Cu at (202.0, 122.0)
- added U6: BGT60UTR13DAiP, BGT60UTR13DAiP:BGT60UTR13DAiP, F.Cu at (177.0, 127.0)
- added U7: TXU0304, Package_SO:TSSOP-14_4.4x5mm_P0.65mm, F.Cu at (180.5, 103.5)
- added U8: TXU0304, Package_SO:TSSOP-14_4.4x5mm_P0.65mm, F.Cu at (180.5, 109.0)
- added U9: KC2016Z80.0000, Oscillator:Oscillator_SMD_Kyocera_KC2520Z-4Pin_2.5x2.0mm, F.Cu at (217.4, 120.7)
- J2: value J3026G01DNLT -> FS USB; footprint J3026G01DNLT:PE_J3026G01DNLT -> Connector_USB:USB_C_Receptacle_GCT_USB4105-xx-A_16P_TopMnt_Horizontal
- moved R5 87.1 mm to (226.4, 77.4), turned to 0 degrees
- moved C1 78.6 mm to (222.4, 69.8), turned to 0 degrees
- moved R6 74.2 mm to (230.5, 69.8), turned to 0 degrees
- moved C2 63.8 mm to (246.5, 84.0)
- moved C3 63.8 mm to (246.5, 86.5)
- moved C4 63.8 mm to (246.5, 89.0)
- moved C5 63.8 mm to (246.5, 91.5)
- moved R7 63.8 mm to (246.5, 94.0)
- moved R10 63.8 mm to (250.5, 89.0)
- moved R11 63.8 mm to (250.5, 91.5)
- moved R12 63.8 mm to (250.5, 94.0)
- moved R8 63.8 mm to (250.5, 84.0)
- moved R9 63.8 mm to (250.5, 86.5)
- moved C6 57.3 mm to (222.4, 72.4)
- moved R2 54.8 mm to (226.4, 69.8)
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Connections:
- net /MCU/ETH_LED2 renamed /Connectors/ETH_LED2
- net /MCU/SWCLK renamed /Portenta/SWCLK
- net /MCU/SWDIO renamed /Portenta/SWDIO
- net /MCU/SWO renamed /Portenta/SWO
- net /MCU/UART0_RX renamed /Portenta/UART4_RX
- net /MCU/UART0_TX renamed /Portenta/UART4_TX
- net /MCU/nRST renamed /Portenta/nRST
- J2 pad S1: GND -> /Connectors/USB_Shield
- R1 pad 2: /MCU/ETH_B- -> /Connectors/ETH_A+
- R10 pad 2: /MCU/I2C1_SDA -> /Portenta/I2C3_SDA
- R11 pad 2: /MCU/I2C1_SCL -> /Portenta/I2C3_SCL
- R2 pad 2: /MCU/ETH_B+ -> /Connectors/ETH_A-
- R3 pad 2: /MCU/ETH_A+ -> /Connectors/ETH_B+
- R4 pad 2: /MCU/ETH_A- -> /Connectors/ETH_B-
- R5 pad 2: Net-(J2-Pad1) -> Net-(J4-Pad1)
- R6 pad 2: Net-(J2-Pad12) -> Net-(J4-Pad12)
- R7 pad 1: /MCU/TOF_RST -> /Portenta/TOF_RST
- R8 pad 2: /MCU/TOF_LPn -> /Portenta/TOF_LPn
- R9 pad 2: /MCU/TOF_INT -> /Portenta/TOF_INT
- U1 pad J1_1: /MCU/ETH_A+ -> /Connectors/ETH_A+
- U1 pad J1_17: /MCU/ETH_LED1 -> /Connectors/ETH_LED1
- U1 pad J1_21: Net-(U1A-VIN-PadJ1_21) -> unconnected-(U1A-VIN-PadJ1_21)
- U1 pad J1_26: /MCU/USB_FS+ -> /Connectors/USB_FS+
- U1 pad J1_28: /MCU/USB_FS- -> /Connectors/USB_FS-
- U1 pad J1_3: /MCU/ETH_A- -> /Connectors/ETH_A-
- U1 pad J1_32: Net-(U1A-VIN-PadJ1_21) -> unconnected-(U1A-VIN-PadJ1_21)
- U1 pad J1_35: /MCU/TOF_LPn -> unconnected-(U1A-UART1_RX-PadJ1_35)
- U1 pad J1_37: /MCU/TOF_RST -> /Camera/CAM_PWDN
- U1 pad J1_39: /MCU/TOF_INT -> /Camera/CAM_nRST
- U1 pad J1_41: Net-(U1A-VIN-PadJ1_21) -> unconnected-(U1A-VIN-PadJ1_21)
- U1 pad J1_43: /MCU/I2C1_SDA -> /Camera/I2C1_SDA
- U1 pad J1_44: /Camera/I2C3_SDA -> /Portenta/I2C3_SDA
- U1 pad J1_45: /MCU/I2C1_SCL -> /Camera/I2C1_SCL
- U1 pad J1_46: /Camera/I2C3_SCL -> /Portenta/I2C3_SCL
- U1 pad J1_48: Net-(U1A-VIN-PadJ1_21) -> unconnected-(U1A-VIN-PadJ1_21)
- U1 pad J1_5: /MCU/ETH_B+ -> /Connectors/ETH_B+
- U1 pad J1_53: Net-(U1A-VSYS-PadJ1_53) -> unconnected-(U1A-VSYS-PadJ1_53)
- U1 pad J1_56: unconnected-(U1A-I2S_MCK-PadJ1_56) -> /Portenta/TOF_RST
- U1 pad J1_58: unconnected-(U1A-I2S_WS-PadJ1_58) -> /Portenta/TOF_INT
- U1 pad J1_60: unconnected-(U1A-I2S_DI-PadJ1_60) -> /Portenta/TOF_LPn
- U1 pad J1_64: Net-(U1A-VSYS-PadJ1_53) -> unconnected-(U1A-VSYS-PadJ1_53)
- U1 pad J1_7: /MCU/ETH_B- -> /Connectors/ETH_B-
- U1 pad J2_26: /MCU/RADAR_INT -> /Portenta/RADAR_INT
- U1 pad J2_28: /MCU/RADAR_RST -> /Portenta/RADAR_RST
- U1 pad J2_36: /MCU/SPI2_NSS -> /Portenta/SPI2_NSS
- U1 pad J2_38: /MCU/SPI2_SCK -> /Portenta/SPI2_SCK
- U1 pad J2_40: /MCU/SPI2_MISO -> /Portenta/SPI2_MISO
- U1 pad J2_42: /MCU/SPI2_MOSI -> /Portenta/SPI2_MOSI
- U2 pad A1: /MCU/TOF_RST -> /Portenta/TOF_RST
- U2 pad A3: /MCU/TOF_INT -> /Portenta/TOF_INT
- U2 pad A5: /MCU/TOF_LPn -> /Portenta/TOF_LPn
- U2 pad C3: /MCU/I2C1_SDA -> /Portenta/I2C3_SDA
- U2 pad C4: /MCU/I2C1_SCL -> /Portenta/I2C3_SCL

Commit message: Finished routing
Parts:
- removed the C18 at (201.4, 103.4)
- removed the C19 at (201.4, 105.9)
- removed the C6 at (222.4, 72.4)
- removed the J2 at (129.0, 90.0)
- removed the U12 at (201.6, 86.9)
- removed the U5 at (202.0, 122.0)
- added C26: 10u, Capacitor_SMD:C_0603_1608Metric, F.Cu at (161.5, 98.7)
- added C27: 10u, Capacitor_SMD:C_0603_1608Metric, F.Cu at (154.7, 97.8)
- added C32: 10u, Capacitor_SMD:C_0603_1608Metric, F.Cu at (155.0, 131.4)
- added C35: 22p, Capacitor_SMD:C_0402_1005Metric, F.Cu at (138.0, 126.8)
- added C38: 10u, Capacitor_SMD:C_0603_1608Metric, F.Cu at (144.4, 113.1)
- added C46: 10u, Capacitor_SMD:C_0603_1608Metric, B.Cu at (149.0, 114.0)
- added C47: 10u, Capacitor_SMD:C_0603_1608Metric, B.Cu at (145.5, 116.6)
- added C48: 10u, Capacitor_SMD:C_0603_1608Metric, B.Cu at (145.5, 118.2)
- added C49: 100n, Capacitor_SMD:C_0603_1608Metric, F.Cu at (142.8, 96.1)
- added C50: 10u, Capacitor_SMD:C_0603_1608Metric, F.Cu at (142.8, 97.8)
- added C55: 100n, Capacitor_SMD:C_0402_1005Metric, F.Cu at (143.5, 104.0)
- added C57: 100n, Capacitor_SMD:C_0603_1608Metric, F.Cu at (153.5, 117.0)
- added C58: 100n, Capacitor_SMD:C_0603_1608Metric, F.Cu at (153.5, 115.0)
- added C59: 100n, Capacitor_SMD:C_0603_1608Metric, F.Cu at (159.5, 117.0)
- added C60: 100n, Capacitor_SMD:C_0603_1608Metric, F.Cu at (159.5, 115.2)
- added C61: 10u, Capacitor_SMD:C_0603_1608Metric, F.Cu at (154.7, 99.6)
- added J3: 1140084168, 1140084168:AMPHENOL_1140084168, B.Cu at (142.4, 95.0)
- added J4: FS USB, 216989-0001:MOLEX_216989-0001, F.Cu at (160.5, 76.0)
- added JP2: 3v3 Select, Jumper:SolderJumper-2_P1.3mm_Open_RoundedPad1.0x1.5mm, B.Cu at (141.7, 109.9)
- added L8: ASPI-4030S-100M-T, Inductor_SMD:L_Abracon_ASPI-4030S, B.Cu at (141.5, 114.5)
- added R10: 2k2, Resistor_SMD:R_0603_1608Metric, B.Cu at (148.8, 104.5)
- added R11: 2k2, Resistor_SMD:R_0603_1608Metric, B.Cu at (148.8, 106.2)
- added U4: TLV74318 SOT23-5, Package_TO_SOT_SMD:SOT-23-5, F.Cu at (158.5, 98.7)
- C14: renamed from C33; moved to B.Cu
- C16: renamed from C38; moved to B.Cu
- C18: renamed from C26; moved to B.Cu
- C19: renamed from C27; moved to B.Cu
- C2: renamed from C21; moved to B.Cu
- C20: renamed from C28; moved to B.Cu
- C21: renamed from C36; moved to B.Cu
- C25: renamed from C42; footprint Capacitor_SMD:C_0603_1608Metric -> Capacitor_SMD:C_0402_1005Metric
- C29: renamed from C3; footprint Capacitor_SMD:C_0603_1608Metric -> Capacitor_SMD:C_0402_1005Metric
- C30: renamed from C4; footprint Capacitor_SMD:C_0603_1608Metric -> Capacitor_SMD:C_0402_1005Metric
- C31: renamed from C5; footprint Capacitor_SMD:C_0603_1608Metric -> Capacitor_SMD:C_0402_1005Metric
- C33: renamed from C8; footprint Capacitor_SMD:C_0603_1608Metric -> Capacitor_SMD:C_0402_1005Metric
- C34: renamed from C7; moved to B.Cu
- C39: renamed from C11; footprint Capacitor_SMD:C_0603_1608Metric -> Capacitor_SMD:C_0402_1005Metric
- C40: renamed from C10; footprint Capacitor_SMD:C_0603_1608Metric -> Capacitor_SMD:C_0402_1005Metric
- C41: renamed from C9; footprint Capacitor_SMD:C_0603_1608Metric -> Capacitor_SMD:C_0402_1005Metric
- C44: value 100n -> 10u
- C45: value 100n -> 1u
- C53: renamed from C46; moved to B.Cu
- C54: renamed from C16; moved to B.Cu
- FB1: footprint Capacitor_SMD:C_0603_1608Metric -> Inductor_SMD:L_0402_1005Metric
- J1: footprint Connector_PinHeader_1.27mm:PinHeader_2x07_P1.27mm_Vertical_SMD -> STDC14_header:PinHeader_2x07_P1.27mm_Vertical_SMD
- JP1, L5, R7: moved to B.Cu
- L6: renamed from L3; moved to B.Cu
- L7: renamed from L6; moved to B.Cu
- R1: renamed from R18; footprint Resistor_SMD:R_0603_1608Metric -> Resistor_SMD:R_0402_1005Metric
- R16: renamed from R15; moved to B.Cu
- R17: renamed from R16; moved to B.Cu
- R18: renamed from R5; moved to B.Cu
- R19: renamed from R6; moved to B.Cu
- R20: renamed from R17; moved to B.Cu
- R4: renamed from R9; moved to B.Cu
- R5: renamed from R8; moved to B.Cu
- R8: renamed from R13; moved to B.Cu
- R9: renamed from R14; moved to B.Cu
- TP1: renamed from TP3; footprint TestPoint:TestPoint_Pad_D1.5mm -> TestPoint:TestPoint_Pad_D1.0mm; moved to B.Cu
- TP2: renamed from TP1; footprint TestPoint:TestPoint_Pad_D1.5mm -> TestPoint:TestPoint_Pad_D1.0mm
- TP3: renamed from TP2; footprint TestPoint:TestPoint_Pad_D1.5mm -> TestPoint:TestPoint_Pad_D1.0mm
- U1: value ABX00042 -> DF40HC(3.5)-80DS-0.4V(51); footprint Portenta:MODULE_ABX00042 -> Portenta:MODULE_ABX00042_NOSCREWS; moved to B.Cu
- U11: value USBLC6-2SC6 -> LM3670MFX-3.3; footprint Package_TO_SOT_SMD:SOT-23-6 -> Package_TO_SOT_SMD:TSOT-23-5; moved to B.Cu
- U12: renamed from U13; moved to B.Cu
- U2: renamed from U9; footprint Oscillator:Oscillator_SMD_Kyocera_KC2520Z-4Pin_2.5x2.0mm -> KC2016Z:KC2016Z
- U3: renamed from U7; moved to B.Cu
- U6: renamed from U8; moved to B.Cu
- U8: renamed from U10; footprint Oscillator:Oscillator_SMD_Kyocera_KC2520Z-4Pin_2.5x2.0mm -> KC2016Z:KC2016Z
- moved R4 111.5 mm to (139.0, 83.3)
- moved R5 111.5 mm to (139.0, 85.0)
- moved C30 109.1 mm to (139.0, 107.5), turned to -90 degrees
- moved R2 109.0 mm to (142.2, 103.5), turned to -90 degrees
- moved R7 108.2 mm to (139.0, 81.6), turned to 180 degrees
- moved C28 107.7 mm to (140.6, 103.5), turned to 90 degrees
- moved R3 106.7 mm to (144.8, 103.5), turned to -90 degrees
- moved R6 104.5 mm to (146.4, 103.5), turned to -90 degrees
- moved C31 104.5 mm to (143.5, 109.2)
- moved FB1 102.6 mm to (138.0, 116.5), turned to -90 degrees
- moved C29 101.7 mm to (147.0, 107.5), turned to -90 degrees
- moved C39 99.5 mm to (138.0, 119.4), turned to 90 degrees
- moved R9 97.7 mm to (147.4, 76.5), turned to 180 degrees
- moved C36 96.3 mm to (139.5, 110.5)
- moved C41 95.5 mm to (138.0, 124.1), turned to -90 degrees
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- renumbered C20 to C1, C17 to C10, C23 to C11, C24 to C12, C25 to C13, C34 to C15, C39 to C17, C37 to C22, C40 to C23, C41 to C24, C2 to C28, C22 to C3, C13 to C36, C12 to C37, C29 to C4, C14 to C42, C15 to C43, C30 to C5, C1 to C51, C31 to C6, C32 to C7, C35 to C8, C43 to C9, J3 to J2, J4 to J5, L4 to L2, L7 to L3, L2 to L4, R1 to R12, R2 to R13, R3 to R14, R4 to R15, R11 to R2, R10 to R3, R12 to R6, U4 to U10, U6 to U5, U2 to U7, U3 to U9
Connections:
- net Net-(U2-RSVD6) renamed /ToF Sensor/RSVD6
- net Net-(U9-CLK) renamed /Radar/80mhz
- C36 pad 1: +3.3V -> +3.3VP
- C42 pad 1: +3.3V -> +3.3VP
- C44 pad 1: +3.3V -> +1V5
- C45 pad 1: +3.3V -> +1V5
- C53 pad 1: +3.3V -> Net-(U12-VBUS)
- J5 pad 11: /Connectors/ETH_LED1 -> Net-(J5-Pad11)
- J5 pad 12: Net-(J4-Pad12) -> +3.3V
- JP1 pad 3: +3.3V -> +3.3VP
- R19 pad 1: +3.3V -> /Connectors/ETH_LED1
- R19 pad 2: Net-(J4-Pad12) -> Net-(J5-Pad11)
- U1 pad J1_23: unconnected-(U1A-USB1_VBUS-PadJ1_23) -> +5V
- U1 pad J1_38: unconnected-(U1A-UART0_RTS-PadJ1_38) -> /Portenta/SDC_CD
- U1 pad J1_55: unconnected-(U1A-SDC_CLK-PadJ1_55) -> /Portenta/SDC_CLK
- U1 pad J1_57: unconnected-(U1A-SDC_CMD-PadJ1_57) -> /Portenta/SDC_CMD
- U1 pad J1_59: unconnected-(U1A-SDC_D0-PadJ1_59) -> /Portenta/SDC_D0
- U1 pad J1_61: unconnected-(U1A-SDC_D1-PadJ1_61) -> /Portenta/SDC_D1
- U1 pad J1_63: unconnected-(U1A-SDC_D2-PadJ1_63) -> /Portenta/SDC_D2
- U1 pad J1_65: unconnected-(U1A-SDC_D3-PadJ1_65) -> /Portenta/SDC_D3
- U1 pad J1_72: unconnected-(U1A-V-SDCARD-PadJ1_72) -> +3.3V
- U1 pad J2_28: /Portenta/RADAR_RST -> /Portenta/RADAR_nRST
- U10 pad 1: +3.3V -> +3.3VP
- U10 pad 3: +3.3V -> +3.3VP
- U11 pad 1: /Connectors/ETH_B- -> +5V
- U11 pad 3: /Connectors/ETH_B+ -> +5V
- U11 pad 4: /Connectors/ETH_B+ -> +3.3VP
- U11 pad 5: +3.3V -> /Camera/LX
- U12 pad 1: /Connectors/USB_FS- -> /Connectors/conn_USB+
- U12 pad 3: /Connectors/USB_FS+ -> /Connectors/conn_USB-
- U12 pad 5: +3.3V -> Net-(U12-VBUS)
- U3 pad 10: /Radar/MISO_1V8 -> /Radar/INT_1V8
- U3 pad 11: /Radar/MOSI_1V8 -> /Radar/SCK_1V8
- U3 pad 12: /Radar/NSS_1V8 -> /Radar/MOSI_1V8
- U3 pad 13: /Radar/SCK_1V8 -> unconnected-(U3-B1Y-Pad13)
- U3 pad 2: /Portenta/SPI2_SCK -> unconnected-(U3-A1-Pad2)
- U3 pad 3: /Portenta/SPI2_NSS -> /Portenta/SPI2_MOSI
- U3 pad 4: /Portenta/SPI2_MOSI -> /Portenta/SPI2_SCK
- U3 pad 5: /Portenta/SPI2_MISO -> /Portenta/RADAR_INT
- U3 pad 7: unconnected-(U7-GND-Pad7) -> GND
- U3 pad 8: +3.3V -> +1V8
- U6 pad 10: /Radar/INT_1V8 -> /Radar/MISO_1V8
- U6 pad 11: unconnected-(U8-B3Y-Pad11) -> /Radar/RST_1V8
- U6 pad 12: unconnected-(U8-B2Y-Pad12) -> /Radar/NSS_1V8
- U6 pad 13: /Radar/RST_1V8 -> unconnected-(U6-B1Y-Pad13)
- U6 pad 2: /Portenta/RADAR_RST -> unconnected-(U6-A1-Pad2)
- U6 pad 3: unconnected-(U8-A2-Pad3) -> /Portenta/SPI2_NSS
- U6 pad 4: unconnected-(U8-A3-Pad4) -> /Portenta/RADAR_nRST
- U6 pad 5: /Portenta/RADAR_INT -> /Portenta/SPI2_MISO
- U6 pad 7: unconnected-(U8-GND-Pad7) -> GND
- U6 pad 8: +3.3V -> +1V8
- U9 pad 1: +3.3V -> +3.3VP
- U9 pad 3: +3.3V -> +3.3VP
Routing:
- net GND: track 0.00 -> 88.8 mm, vias 0 -> 114
- net /Camera/CAM_PWDN: track 0.00 -> 57.4 mm, vias 0 -> 3
- net +3.3V: track 0.00 -> 56.5 mm, vias 0 -> 26
- net /Camera/CAM_nRST: track 0.00 -> 50.5 mm, vias 0 -> 4
- net VD: track 0.00 -> 49.9 mm, vias 0 -> 1
- net +5V: track 0.00 -> 43.6 mm, vias 0 -> 2
- net /Camera/I2C1_SDA: track 0.00 -> 42.8 mm, vias 0 -> 3
- net /Camera/I2C1_SCL: track 0.00 -> 42.8 mm, vias 0 -> 3
- net +3.3VP: track 0.00 -> 40.3 mm, vias 0 -> 1
- net /Portenta/TOF_RST: track 0.00 -> 37.4 mm, vias 0 -> 3
- net /Portenta/TOF_INT: track 0.00 -> 34.5 mm, vias 0 -> 3
- net /Portenta/TOF_LPn: track 0.00 -> 32.0 mm, vias 0 -> 2
- net /Portenta/SWO: track 0.00 -> 30.3 mm, vias 0 -> 1
- net +1V8: track 0.00 -> 29.9 mm, vias 0 -> 9
- net /Portenta/I2C3_SCL: track 0.00 -> 29.3 mm, vias 0 -> 2
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- added copper zone on In2.Cu, net +1V8
- added copper zone on In3.Cu, net +3.3V
- added copper zone on B.Cu, net +3.3VP
- added copper zone on B.Cu, net /Camera/LX
- added copper zone on F.Cu, net GND
- added copper zone on In1.Cu, net GND
- added copper zone on In4.Cu, net GND
Other:
- board size 66 x 66 mm -> 25.4 x 66 mm
- copper layers 2 -> 6
- board text added: "60.9°"
- board text added: "63.2°"
- board text added: "Signals - layer assignment: Radar SPI - Bottom signal Camera - Inner signal ToF - Inner signal Ethernet - Top signal FS USB - Bottom signal microSD - Bottom signal"
- board text added: "↑"
- board text added: "↓"
