File: hardware/camera.kicad_sch (KiCad schematic)
At the start: 20 parts, among them J3 Camera, U3 TLV74328 SOT23-5, U4 TLV74315 SOT23-5, X1 OSC-24MHz

Commit message: final-ish schematic
Parts:
- removed X1: OSC-24MHz, Oscillator:Oscillator_SMD_ECS_2520MV-xxx-xx-4Pin_2.5x2.0mm, symbol Oscillator:ECS-2520MV-xxx-xx
- added U9: KC2016Z24.0000, Oscillator:Oscillator_SMD_Kyocera_KC2520Z-4Pin_2.5x2.0mm, symbol Oscillator:KC2520Z
- C10, C11, C12, C13, C14, C15, C7, C8, C9, FB1: footprint (none) -> Capacitor_SMD:C_0603_1608Metric
- J3: footprint (none) -> OV5640:OV2640FSL; symbol Connector_Generic_MountingPin:Conn_01x24_MountingPin -> Connector_Generic:Conn_01x24
- JP1: footprint (none) -> Jumper:SolderJumper-3_P1.3mm_Open_RoundedPad1.0x1.5mm
- R13, R14: footprint (none) -> Resistor_SMD:R_0603_1608Metric
- TP1, TP2, TP3: footprint (none) -> TestPoint:TestPoint_Pad_D1.5mm
Connections:
- net GND: now also U9.2 (GND)
- net VD: now also U9.1 (INH), U9.4 (VCC)
- net XCLK: now also U9.3 (CLK)
- no-connect marks 1 -> 0
Other:
- note added: "I_{max} = 180mA"
- note added: "I_{max} = 7.3mA"

Commit message: Finished routing
Parts:
- added C32, C38, C44, C46, C47, C48: 10u, Capacitor_SMD:C_0603_1608Metric, symbol Device:C
- added C35: 22p, Capacitor_SMD:C_0402_1005Metric, symbol Device:C
- added C45: 1u, Capacitor_SMD:C_0603_1608Metric, symbol Device:C
- added JP2: 3v3 Select, Jumper:SolderJumper-2_P1.3mm_Open_RoundedPad1.0x1.5mm, symbol Jumper:SolderJumper_2_Open
- added L8: ASPI-4030S-100M-T, Inductor_SMD:L_Abracon_ASPI-4030S, symbol Device:L
- added R10, R11: 2k2, Resistor_SMD:R_0603_1608Metric, symbol Device:R
- added U5: LM3670MFX-3.3, Package_TO_SOT_SMD:TSOT-23-5, symbol Regulator_Switching:LM3670MF
- C33: renamed from C8; footprint Capacitor_SMD:C_0603_1608Metric -> Capacitor_SMD:C_0402_1005Metric
- C39: renamed from C11; footprint Capacitor_SMD:C_0603_1608Metric -> Capacitor_SMD:C_0402_1005Metric
- C40: renamed from C10; footprint Capacitor_SMD:C_0603_1608Metric -> Capacitor_SMD:C_0402_1005Metric
- C41: renamed from C9; footprint Capacitor_SMD:C_0603_1608Metric -> Capacitor_SMD:C_0402_1005Metric
- FB1: footprint Capacitor_SMD:C_0603_1608Metric -> Inductor_SMD:L_0402_1005Metric
- TP1: renamed from TP3; footprint TestPoint:TestPoint_Pad_D1.5mm -> TestPoint:TestPoint_Pad_D1.0mm
- TP2: renamed from TP1; footprint TestPoint:TestPoint_Pad_D1.5mm -> TestPoint:TestPoint_Pad_D1.0mm
- TP3: renamed from TP2; footprint TestPoint:TestPoint_Pad_D1.5mm -> TestPoint:TestPoint_Pad_D1.0mm
- U9: footprint Oscillator:Oscillator_SMD_Kyocera_KC2520Z-4Pin_2.5x2.0mm -> KC2016Z:KC2016Z
- renumbered C7 to C34, C13 to C36, C12 to C37, C14 to C42, C15 to C43, J3 to J2, R13 to R8, R14 to R9, U4 to U10, U3 to U9
Connections:
- net +1V5: now also C44.1, C45.1
- net +2V8: now also C38.1
- net +3.3V: now also JP2.2 (B); no longer C36.1, C42.1, JP1.3 (B), U10.1 (IN), U10.3 (EN), U9.1 (IN), U9.3 (EN)
- net CAM_CK: now also C35.1
- net GND: now also C32.2, C35.2, C38.2, C44.2, C45.2, C46.2, C47.2, C48.2, U5.2 (GND)
- net I2C1_SCL: now also R11.2
- net I2C1_SDA: now also R10.2
- net VD: now also C32.1, R10.1, R11.1
- new net +3.3VP: C36.1, C42.1, C47.1, C48.1, JP1.3 (B), JP2.1 (A), L8.2, U10.1 (IN), U10.3 (EN), U5.4 (FB), U9.1 (IN), U9.3 (EN)
- new net +5V: C46.1, U5.1 (Vin), U5.3 (EN)
- new net LX: L8.1, U5.5 (SW)
Other:
- note added: "I_{max} = 190mA"
- moved on the sheet: C39, C40, C41, R9

Commit message: Add testpoints, 0ohm, led, logos
Parts:
- removed JP1: VIO Select, Jumper:SolderJumper-3_P1.3mm_Open_RoundedPad1.0x1.5mm, symbol Jumper:SolderJumper_3_Open
- added R21: 0, Resistor_SMD:R_0603_1608Metric, symbol Device:R
- added TP15: SDA1, TestPoint:TestPoint_Pad_D1.0mm, symbol Connector:TestPoint
- added TP16: SCL1, TestPoint:TestPoint_Pad_D1.0mm, symbol Connector:TestPoint
Connections:
- net VD is gone; now on net VCAM: C32.1, C33.1, C41.1, J2.11 (Pin_11), R10.1, R11.1, R8.1, U9.1 (INH), U9.4 (VCC)
- net +5V: now also R21.1; no longer C46.1, U5.1 (Vin), U5.3 (EN)
- net I2C1_SCL: now also TP16.1
- net I2C1_SDA: now also TP15.1
- net +3.3VP renamed VCAM
- new net 5v_tof: C46.1, R21.2, U5.1 (Vin), U5.3 (EN)

Commit message: Final fixes, manufacturing
Parts:
- C32, C36, C37, C38, C42, C43, C44, C46, C47, C48: MANUFACTURER (none) -> Murata; MOUSER NO (none) -> 81-GRM188Z71A106KA3D; PART NO (none) -> GRM188Z71A106KA73D
- C33, C39, C40, C41: MANUFACTURER (none) -> Murata; MOUSER NO (none) -> 81-GRM155R71H104KE4D; PART NO (none) -> GRM155R71H104KE14D
- C34: MANUFACTURER (none) -> KEMET; MOUSER NO (none) -> 80-C603C104K5RAC3121; PART NO (none) -> C0603C104K5RAC3121
- C35: MANUFACTURER (none) -> Murata; MOUSER NO (none) -> 81-GCM1555C1H220JA6J; PART NO (none) -> GCM1555C1H220JA16J
- C45: MANUFACTURER (none) -> Murata; MOUSER NO (none) -> 81-GCJ188R71E105KA1D; PART NO (none) -> GCJ188R71E105KA01D
- J2: MANUFACTURER (none) -> Hirose; MOUSER NO (none) -> 798-FH12-24S-0.5SH55; PART NO (none) -> FH12-24S-0.5SH(55)
- L8: value ASPI-4030S-100M-T -> 74438336022; footprint Inductor_SMD:L_Abracon_ASPI-4030S -> Inductor_SMD:L_Wuerth_MAPI-3020; MANUFACTURER (none) -> Wuerth; MOUSER NO (none) -> 710-74438336022; PART NO (none) -> 74438336022
- L9: renamed from FB1; value FerriteBead -> BLM15PX471SZ1D; symbol Device:FerriteBead -> Device:L; MANUFACTURER (none) -> Murata; MOUSER NO (none) -> 81-BLM15PX471SZ1D; PART NO (none) -> BLM15PX471SZ1D
- R10, R11: MANUFACTURER (none) -> Vishay / Dale; MOUSER NO (none) -> 71-CRCW06032K20FKEAC; PART NO (none) -> CRCW06032K20FKEAC
- R21: MANUFACTURER (none) -> Vishay / Dale; MOUSER NO (none) -> 71-CRCW06030000Z0EBC; PART NO (none) -> CRCW06030000Z0EBC
- R8, R9: MANUFACTURER (none) -> Vishay / Dale; MOUSER NO (none) -> 71-CRCW060310K0FKEAC; PART NO (none) -> CRCW060310K0FKEAC
- U10: MANUFACTURER (none) -> Texas Instruments; MOUSER NO (none) -> 595-TLV74315PDBVR; PART NO (none) -> TLV74315PDBVR
- U5: value LM3670MFX-3.3 -> LM3671MF-3.3; MANUFACTURER (none) -> Texas Instruments; MOUSER NO (none) -> 926-LM3671MF-3.3NOPB; PART NO (none) -> LM3671MF-3.3/NOPB
- U9: MANUFACTURER (none) -> KYOCERA AVX; MOUSER NO (none) -> 581-KC2016Z240C1KX00; PART NO (none) -> KC2016Z24.0000C1KX00
- U9: MANUFACTURER (none) -> Texas Instruments; MOUSER NO (none) -> 595-TLV74328PDBVR; PART NO (none) -> TLV74328PDBVR
