File: hardware/conn.kicad_sch (KiCad schematic)
At the start: 14 parts, among them J2 J3026G01DNLT, J4 FS USB

Commit message: final-ish schematic
Parts:
- added C1 (x3): 100n, Capacitor_SMD:C_0603_1608Metric, symbol Device:C
- added U11, U12, U13: USBLC6-2SC6, Package_TO_SOT_SMD:SOT-23-6, symbol Power_Protection:USBLC6-2SC6
- C16: footprint (none) -> Capacitor_SMD:C_0603_1608Metric
- J4: footprint (none) -> Connector_USB:USB_C_Receptacle_GCT_USB4105-xx-A_16P_TopMnt_Horizontal
- R15, R16, R17: footprint (none) -> Resistor_SMD:R_0603_1608Metric
Connections:
- net +3.3V: now also C1.1, C1.1, C1.1, U11.5 (VBUS), U12.5 (VBUS), U13.5 (VBUS)
- net ETH_A+: now also U12.3 (I/O2), U12.4 (I/O2)
- net ETH_A-: now also U12.1 (I/O1), U12.6 (I/O1)
- net ETH_B+: now also U11.3 (I/O2), U11.4 (I/O2)
- net ETH_B-: now also U11.1 (I/O1), U11.6 (I/O1)
- net GND: now also C1.2, C1.2, C1.2, U11.2 (GND), U12.2 (GND), U13.2 (GND)
- net USB_FS+: now also U13.3 (I/O2), U13.4 (I/O2)
- net USB_FS-: now also U13.1 (I/O1), U13.6 (I/O1)
Other:
- note added: "Place TVS array inline"
- note added: "Place TVS arrays inline"
- note removed: "TODO: ESD protection"
- company: (none) -> Center for Project-Based Learning
- title: (none) -> Heterogeneous radar, RGB, and ToF sensor board
- moved on the sheet: C1, C16, C6, J2, J4, R1, R15, R16, R17, R2, R3, R4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

Commit message: Finished routing
Parts:
- removed C1 (x2), C6: 100n, Capacitor_SMD:C_0603_1608Metric, symbol Device:C
- removed U11, U12: USBLC6-2SC6, Package_TO_SOT_SMD:SOT-23-6, symbol Power_Protection:USBLC6-2SC6
- J4: footprint Connector_USB:USB_C_Receptacle_GCT_USB4105-xx-A_16P_TopMnt_Horizontal -> 216989-0001:MOLEX_216989-0001
- renumbered C16 to C54, R15 to R16, R16 to R17, R17 to R20, U13 to U12
Connections:
- net +3.3V: now also J2.12; no longer C1.1, R6.1, U12.5 (VBUS)
- net ETH_LED1: now also R6.1; no longer J2.11
- net USB_FS+: no longer J4.A6 (D+), J4.B6 (D+), U12.3 (I/O2)
- net USB_FS-: no longer J4.A7 (D-), J4.B7 (D-), U12.1 (I/O1)
- net at R6.2: now also J2.11; no longer J2.12
- new net: C1.1, U12.5 (VBUS)
- new net conn_USB+: J4.A7 (D-), J4.B7 (D-), U12.1 (I/O1)
- new net conn_USB-: J4.A6 (D+), J4.B6 (D+), U12.3 (I/O2)
Other:
- note removed: "Place TVS arrays inline"
- moved on the sheet: C1, C54, J2, J4, R1, R16, R17, R2, R20, R3, R4, R5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

Commit message: Final fixes, manufacturing
Parts:
- C1: MANUFACTURER (none) -> KEMET; MOUSER NO (none) -> 80-C603C104K5RAC3121; PART NO (none) -> C0603C104K5RAC3121
- C54: MANUFACTURER (none) -> KEMET; MOUSER NO (none) -> 80-C0603V102KDR; PART NO (none) -> C0603V102KDRACTU
- J2: MOUSER NO (none) -> 673-J3026G01DNL; PART NO (none) -> J3026G01DNL
- J4: MANUFACTURER (none) -> Molex; MOUSER NO (none) -> 538-216989-0001; PART NO (none) -> 216989-0001
- R1, R2, R3, R4: MANUFACTURER (none) -> Vishay / Dale; MOUSER NO (none) -> 71-CRCW060349R9FKEAC; PART NO (none) -> CRCW060349R9FKEAC
- R16, R17: MANUFACTURER (none) -> Vishay / Dale; MOUSER NO (none) -> 71-CRCW06035K10FKEAC; PART NO (none) -> CRCW06035K10FKEAC
- R20: MANUFACTURER (none) -> Vishay / Dale; MOUSER NO (none) -> 71-CRCW06031M00FKEAC; PART NO (none) -> CRCW06031M00FKEAC
- R5, R6: MANUFACTURER (none) -> Vishay / Dale; MOUSER NO (none) -> 71-CRCW0603470RFKEAC; PART NO (none) -> CRCW0603470RFKEAC
- U12: MANUFACTURER (none) -> STMicroelectronics; MOUSER NO (none) -> 511-USBLC6-2SC6; PART NO (none) -> USBLC6-2SC6
Changed lines of the file:
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@@
   (title_block
     (title "Heterogeneous radar, RGB, and ToF sensor board")
-    (date "2023-04-25")
-    (rev "1.3")
+    (date "2023-04-26")
+    (rev "1.4")
     (company "Center for Project-Based Learning")
     (comment 1 "Zoltán Marcsek")
@@
       (effects (font (size 1.27 1.27)) hide)
     )
-    (property "Datasheet" "~" (at 139.7 144.78 0)
+    (property "Datasheet" "https://www.mouser.ch/datasheet/2/427/crcwce3-1762584.pdf" (at 139.7 144.78 0)
+      (effects (font (size 1.27 1.27)) hide)
+    )
+    (property "MOUSER NO" "71-CRCW0603470RFKEAC" (at 139.7 144.78 0)
+      (effects (font (size 1.27 1.27)) hide)
+    )
+    (property "PART NO" "CRCW0603470RFKEAC" (at 139.7 144.78 0)
+      (effects (font (size 1.27 1.27)) hide)
+    )
+    (property "MANUFACTURER" "Vishay / Dale" (at 139.7 144.78 0)
       (effects (font (size 1.27 1.27)) hide)
     )
@@
       (effects (font (size 1.27 1.27)) hide)
     )
-    (property "Datasheet" "~" (at 121.92 88.9 0)
+    (property "Datasheet" "https://www.mouser.ch/datasheet/2/427/crcwce3-1762584.pdf" (at 121.92 88.9 0)
+      (effects (font (size 1.27 1.27)) hide)
+    )
+    (property "MOUSER NO" "71-CRCW060349R9FKEAC" (at 121.92 88.9 0)
+      (effects (font (size 1.27 1.27)) hide)
+    )
+    (property "PART NO" "CRCW060349R9FKEAC" (at 121.92 88.9 0)
+      (effects (font (size 1.27 1.27)) hide)
+    )
+    (property "MANUFACTURER" "Vishay / Dale" (at 121.92 88.9 0)
       (effects (font (size 1.27 1.27)) hide)
     )
@@
       (effects (font (size 1.27 1.27)) hide)
     )
-    (property "Datasheet" "~" (at 139.7 40.64 0)
+    (property "Datasheet" "https://www.mouser.ch/datasheet/2/427/crcwce3-1762584.pdf" (at 139.7 40.64 0)
+      (effects (font (size 1.27 1.27)) hide)
+    )
+    (property "MOUSER NO" "71-CRCW06035K10FKEAC" (at 139.7 40.64 0)
+      (effects (font (size 1.27 1.27)) hide)
+    )
+    (property "PART NO" "CRCW06035K10FKEAC" (at 139.7 40.64 0)
+      (effects (font (size 1.27 1.27)) hide)
+    )
+    (property "MANUFACTURER" "Vishay / Dale" (at 139.7 40.64 0)
       (effects (font (size 1.27 1.27)) hide)
     )
@@
       (effects (font (size 1.27 1.27)) hide)
     )
-    (property "Datasheet" "~" (at 184.15 68.58 0)
+    (property "Datasheet" "https://www.mouser.ch/datasheet/2/427/crcwce3-1762584.pdf" (at 184.15 68.58 0)
+      (effects (font (size 1.27 1.27)) hide)
+    )
+    (property "MOUSER NO" "71-CRCW06031M00FKEAC" (at 184.15 68.58 0)
+      (effects (font (size 1.27 1.27)) hide)
+    )
+    (property "PART NO" "CRCW06031M00FKEAC" (at 184.15 68.58 0)
+      (effects (font (size 1.27 1.27)) hide)
+    )
+    (property "MANUFACTURER" "Vishay / Dale" (at 184.15 68.58 0)
       (effects (font (size 1.27 1.27)) hide)
     )
@@
       (effects (font (size 1.27 1.27)) hide)
     )
-    (property "Datasheet" "~" (at 129.54 88.9 0)
+    (property "Datasheet" "https://www.mouser.ch/datasheet/2/427/crcwce3-1762584.pdf" (at 129.54 88.9 0)
+      (effects (font (size 1.27 1.27)) hide)
+    )
+    (property "MOUSER NO" "71-CRCW060349R9FKEAC" (at 129.54 88.9 0)
+      (effects (font (size 1.27 1.27)) hide)
+    )
+    (property "PART NO" "CRCW060349R9FKEAC" (at 129.54 88.9 0)
+      (effects (font (size 1.27 1.27)) hide)
+    )
+    (property "MANUFACTURER" "Vishay / Dale" (at 129.54 88.9 0)
       (effects (font (size 1.27 1.27)) hide)
     )
@@
       (effects (font (size 1.27 1.27)) hide)
     )
-    (property "Datasheet" "~" (at 114.3 88.9 0)
+    (property "Datasheet" "https://www.mouser.ch/datasheet/2/427/crcwce3-1762584.pdf" (at 114.3 88.9 0)
+      (effects (font (size 1.27 1.27)) hide)
+    )
+    (property "MOUSER NO" "71-CRCW060349R9FKEAC" (at 114.3 88.9 0)
+      (effects (font (size 1.27 1.27)) hide)
+    )
+    (property "PART NO" "CRCW060349R9FKEAC" (at 114.3 88.9 0)
+      (effects (font (size 1.27 1.27)) hide)
+    )
+    (property "MANUFACTURER" "Vishay / Dale" (at 114.3 88.9 0)
       (effects (font (size 1.27 1.27)) hide)
     )
@@
       (effects (font (size 1.27 1.27)) (justify bottom) hide)
     )
-    (property "Datasheet" "https://eu.mouser.com/datasheet/2/447/J409-2903620.pdf" (at 165.1 127 0)
+    (property "Datasheet" "https://www.mouser.ch/datasheet/2/447/J409-2903620.pdf" (at 165.1 127 0)
       (effects (font (size 1.27 1.27)) hide)
     )
@@
     (property "MAXIMUM_PACKAGE_HEIGHT" "13.86 mm" (at 165.1 127 0)
       (effects (font (size 1.27 1.27)) (justify bottom) hide)
+    )
+    (property "MOUSER NO" "673-J3026G01DNL" (at 165.1 127 0)
+      (effects (font (size 1.27 1.27)) hide)
+    )
+    (property "PART NO" "J3026G01DNL" (at 165.1 127 0)
+      (effects (font (size 1.27 1.27)) hide)
     )
     (pin "1")
@@
       (effects (font (size 1.27 1.27)) hide)
     )
-    (property "Datasheet" "~" (at 139.7 124.46 0)
+    (property "Datasheet" "https://www.mouser.ch/datasheet/2/427/crcwce3-1762584.pdf" (at 139.7 124.46 0)
+      (effects (font (size 1.27 1.27)) hide)
+    )
+    (property "MOUSER NO" "71-CRCW0603470RFKEAC" (at 139.7 124.46 0)
+      (effects (font (size 1.27 1.27)) hide)
+    )
+    (property "PART NO" "CRCW0603470RFKEAC" (at 139.7 124.46 0)
+      (effects (font (size 1.27 1.27)) hide)
+    )
+    (property "MANUFACTURER" "Vishay / Dale" (at 139.7 124.46 0)
       (effects (font (size 1.27 1.27)) hide)
     )
@@
       (effects (font (size 1.27 1.27)) hide)
     )
-    (property "Datasheet" "~" (at 184.15 73.66 0)
+    (property "Datasheet" "https://www.mouser.ch/datasheet/2/212/KEM_C1034_X7R_HV_ARC_SMD-1101730.pdf" (at 184.15 73.66 0)
+      (effects (font (size 1.27 1.27)) hide)
+    )
+    (property "MOUSER NO" "80-C0603V102KDR" (at 184.15 73.66 0)
+      (effects (font (size 1.27 1.27)) hide)
+    )
+    (property "PART NO" "C0603V102KDRACTU" (at 184.15 73.66 0)
+      (effects (font (size 1.27 1.27)) hide)
+    )
+    (property "MANUFACTURER" "KEMET" (at 184.15 73.66 0)
       (effects (font (size 1.27 1.27)) hide)
     )
@@
       (effects (font (size 1.27 1.27)) hide)
     )
-    (property "Datasheet" "~" (at 106.68 88.9 0)
+    (property "Datasheet" "https://www.mouser.ch/datasheet/2/427/crcwce3-1762584.pdf" (at 106.68 88.9 0)
+      (effects (font (size 1.27 1.27)) hide)
+    )
+    (property "MOUSER NO" "71-CRCW060349R9FKEAC" (at 106.68 88.9 0)
+      (effects (font (size 1.27 1.27)) hide)
+    )
+    (property "PART NO" "CRCW060349R9FKEAC" (at 106.68 88.9 0)
+      (effects (font (size 1.27 1.27)) hide)
+    )
+    (property "MANUFACTURER" "Vishay / Dale" (at 106.68 88.9 0)
       (effects (font (size 1.27 1.27)) hide)
     )
@@
       (effects (font (size 1.27 1.27)) hide)
     )
-    (property "Datasheet" "~" (at 142.24 87.63 0)
+    (property "Datasheet" "https://www.mouser.ch/datasheet/2/212/KEM_C1023_X7R_AUTO_SMD-1093309.pdf" (at 142.24 87.63 0)
+      (effects (font (size 1.27 1.27)) hide)
+    )
+    (property "MANUFACTURER" "KEMET" (at 142.24 87.63 0)
+      (effects (font (size 1.27 1.27)) hide)
+    )
+    (property "MOUSER NO" "80-C603C104K5RAC3121" (at 142.24 87.63 0)
+      (effects (font (size 1.27 1.27)) hide)
+    )
+    (property "PART NO" "C0603C104K5RAC3121" (at 142.24 87.63 0)
       (effects (font (size 1.27 1.27)) hide)
     )
@@
       (effects (font (size 1.27 1.27)) hide)
     )
-    (property "Datasheet" "~" (at 82.55 58.42 0)
+    (property "Datasheet" "https://www.mouser.ch/datasheet/2/212/KEM_C1023_X7R_AUTO_SMD-1093309.pdf" (at 82.55 58.42 0)
+      (effects (font (size 1.27 1.27)) hide)
+    )
+    (property "MANUFACTURER" "KEMET" (at 82.55 58.42 0)
+      (effects (font (size 1.27 1.27)) hide)
+    )
+    (property "MOUSER NO" "80-C603C104K5RAC3121" (at 82.55 58.42 0)
+      (effects (font (size 1.27 1.27)) hide)
+    )
+    (property "PART NO" "C0603C104K5RAC3121" (at 82.55 58.42 0)
       (effects (font (size 1.27 1.27)) hide)
     )
@@
     )
     (property "Datasheet" "https://www.st.com/resource/en/datasheet/usblc6-2.pdf" (at 105.41 57.15 0)
+      (effects (font (size 1.27 1.27)) hide)
+    )
+    (property "MOUSER NO" "511-USBLC6-2SC6" (at 114.3 52.07 0)
+      (effects (font (size 1.27 1.27)) hide)
+    )
+    (property "PART NO" "USBLC6-2SC6" (at 114.3 52.07 0)
+      (effects (font (size 1.27 1.27)) hide)
+    )
+    (property "MANUFACTURER" "STMicroelectronics" (at 114.3 52.07 0)
       (effects (font (size 1.27 1.27)) hide)
     )
@@
       (effects (font (size 1.27 1.27)) hide)
     )
-    (property "Datasheet" "https://www.usb.org/sites/default/files/documents/usb_type-c.zip" (at 161.29 50.8 0)
+    (property "Datasheet" "https://www.molex.com/webdocs/datasheets/pdf/en-us/2169890001_IO_CONNECTORS.pdf" (at 161.29 50.8 0)
+      (effects (font (size 1.27 1.27)) hide)
+    )
+    (property "MOUSER NO" "538-216989-0001" (at 165.1 50.8 0)
+      (effects (font (size 1.27 1.27)) hide)
+    )
+    (property "PART NO" "216989-0001" (at 165.1 50.8 0)
+      (effects (font (size 1.27 1.27)) hide)
+    )
+    (property "MANUFACTURER" "Molex" (at 165.1 50.8 0)
       (effects (font (size 1.27 1.27)) hide)
     )
@@
       (effects (font (size 1.27 1.27)) hide)
     )
-    (property "Datasheet" "~" (at 139.7 43.18 0)
-      (effects (font (size 1.27 1.27)) hide)
-    )
+    (property "Datasheet" "https://www.mouser.ch/datasheet/2/427/crcwce3-1762584.pdf" (at 139.7 43.18 0)
+      (effects (font (size 1.27 1.27)) hide)
+    )
+    (property "MOUSER NO" "71-CRCW06035K10FKEAC" (at 139.7 43.18 0)
+      (effects (font (size 1.27 1.27)) hide)
+    )
+    (property "PART NO" "CRCW06035K10FKEAC" (at 139.7 43.18 0)
+      (effects (font (size 1.27 1.27)) hide)
+    )
+    (property "MANUFACTURER" "Vishay / Dale" (at 139.7 43.18 0)
+      (effects (font (size 1.27 1.27)) hide)
+    )
