File: hardware/mcu.kicad_sch (KiCad schematic)
At the start: 2 parts, among them J1 Debug, U1 ABX00042

Commit message: final-ish schematic
Connections:
- now unconnected: U1.J1_11 (NC), U1.J1_13 (NC), U1.J1_15 (NC), U1.J1_2 (NC), U1.J1_24 (NC), U1.J1_30 (NC), U1.J1_4 (NC), U1.J1_50 (NC), U1.J1_52 (NC), U1.J1_6 (NC), U1.J1_67 (NC), U1.J1_69 (NC), U1.J1_70 (NC), U1.J1_71 (NC), U1.J1_74 (NC), U1.J1_76 (NC), U1.J1_78 (NC), U1.J1_8 (NC), U1.J1_80 (NC), U1.J1_9 (NC), U1.J2_11 (NC_1), U1.J2_13 (NC_1), U1.J2_15 (NC_1), U1.J2_17 (NC_1), U1.J2_19 (NC_1), U1.J2_21 (NC_1), U1.J2_29 (NC_1), U1.J2_30 (NC_1), U1.J2_31 (NC_1), U1.J2_32 (NC_1), U1.J2_35 (NC_1), U1.J2_37 (NC_1), U1.J2_39 (NC_1), U1.J2_41 (NC_1), U1.J2_55 (NC_1), U1.J2_9 (NC_1)
- no-connect marks 8 -> 68
Other:
- note added: "Shared with PMIC, crypto"
Changed lines of the file:
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@@
   (title_block
     (title "Heterogeneous radar, RGB, and ToF sensor board")
-    (date "2023-04-12")
+    (date "2023-04-17")
     (rev "0")
     (company "Center for Project-Based Learning")
@@
   (junction (at 76.2 184.15) (diameter 0) (color 0 0 0 0)
   )
+  (no_connect (at 50.8 99.06))
+  (no_connect (at 101.6 73.66))
+  (no_connect (at 190.5 81.28))
+  (no_connect (at 241.3 96.52))
   (no_connect (at 88.9 165.1))
+  (no_connect (at 101.6 43.18))
+  (no_connect (at 241.3 104.14))
+  (no_connect (at 241.3 106.68))
+  (no_connect (at 190.5 78.74))
   (no_connect (at 88.9 170.18))
+  (no_connect (at 190.5 45.72))
+  (no_connect (at 190.5 116.84))
+  (no_connect (at 190.5 119.38))
+  (no_connect (at 190.5 68.58))
+  (no_connect (at 241.3 91.44))
+  (no_connect (at 190.5 40.64))
   (no_connect (at 190.5 58.42))
+  (no_connect (at 190.5 71.12))
+  (no_connect (at 50.8 101.6))
+  (no_connect (at 190.5 88.9))
+  (no_connect (at 50.8 106.68))
+  (no_connect (at 101.6 104.14))
+  (no_connect (at 50.8 104.14))
+  (no_connect (at 50.8 33.02))
   (no_connect (at 50.8 55.88))
+  (no_connect (at 190.5 50.8))
+  (no_connect (at 190.5 38.1))
+  (no_connect (at 190.5 111.76))
+  (no_connect (at 101.6 111.76))
+  (no_connect (at 241.3 88.9))
+  (no_connect (at 190.5 96.52))
+  (no_connect (at 190.5 53.34))
+  (no_connect (at 50.8 71.12))
+  (no_connect (at 241.3 101.6))
+  (no_connect (at 190.5 43.18))
   (no_connect (at 50.8 60.96))
+  (no_connect (at 50.8 109.22))
+  (no_connect (at 190.5 109.22))
+  (no_connect (at 101.6 48.26))
+  (no_connect (at 190.5 104.14))
+  (no_connect (at 190.5 91.44))
+  (no_connect (at 50.8 88.9))
+  (no_connect (at 190.5 93.98))
+  (no_connect (at 50.8 96.52))
+  (no_connect (at 190.5 99.06))
+  (no_connect (at 101.6 40.64))
+  (no_connect (at 101.6 30.48))
+  (no_connect (at 190.5 66.04))
+  (no_connect (at 241.3 99.06))
+  (no_connect (at 190.5 83.82))
   (no_connect (at 50.8 58.42))
+  (no_connect (at 101.6 45.72))
+  (no_connect (at 241.3 93.98))
+  (no_connect (at 50.8 91.44))
+  (no_connect (at 101.6 109.22))
   (no_connect (at 190.5 60.96))
+  (no_connect (at 50.8 68.58))
+  (no_connect (at 190.5 76.2))
+  (no_connect (at 241.3 109.22))
+  (no_connect (at 241.3 111.76))
+  (no_connect (at 101.6 27.94))
+  (no_connect (at 190.5 106.68))
+  (no_connect (at 101.6 76.2))
+  (no_connect (at 101.6 50.8))
   (no_connect (at 50.8 63.5))
+  (no_connect (at 190.5 86.36))
+  (no_connect (at 101.6 38.1))
+  (no_connect (at 190.5 114.3))
   (bus_entry (at 254 38.1) (size -2.54 2.54)
     (stroke (width 0) (type default))
@@
   )
   (text "Camera" (at 271.78 50.8 0)
-    (effects (font (face "AmsiPro-Bold") (size 2.5 2.5)) (justify left bottom))
+    (effects (font (face "Asap") (size 2.5 2.5)) (justify left bottom))
   )
   (text "PI9" (at 127 71.12 0)
     (effects (font (size 1.27 1.27)) (justify left bottom))
+  )
+  (text "Shared with PMIC, crypto" (at 21.59 87.63 0)
+    (effects (font (face "Asap") (size 1.27 1.27)) (justify left bottom))
   )
   (text "PH10" (at 266.7 53.34 0)
@@
   )
   (text "Debug" (at 133.35 71.12 0)
-    (effects (font (face "AmsiPro-Bold") (size 2.5 2.5)) (justify left bottom))
+    (effects (font (face "Asap") (size 2.5 2.5)) (justify left bottom))
   )
   (text "Radar" (at 271.78 77.47 0)
-    (effects (font (face "AmsiPro-Bold") (size 2.5 2.5)) (justify left bottom))
+    (effects (font (face "Asap") (size 2.5 2.5)) (justify left bottom))
   )
   (text "PI4" (at 266.7 43.18 0)
@@
   )
   (text "Debug" (at 20.32 123.19 90)
-    (effects (font (face "AmsiPro-Bold") (size 2.5 2.5)) (justify left bottom))
+    (effects (font (face "Asap") (size 2.5 2.5)) (justify left bottom))
   )
   (text "PI2" (at 127 101.6 0)
@@
     (effects (font (size 1.27 1.27)) (justify left bottom))
   )
-  (text "Camera" (at 20.32 71.12 90)
-    (effects (font (face "AmsiPro-Bold") (size 2.5 2.5)) (justify right bottom))
+  (text "Camera" (at 20.32 72.39 90)
+    (effects (font (face "Asap") (size 2.5 2.5)) (justify right bottom))
   )
   (text "PI15" (at 21.59 76.2 0)
@@
     )
   )
-  (symbol (lib_name "ABX00042_1") (lib_id "ABX00042:ABX00042") (at 76.2 76.2 0) (unit 1)
+  (symbol (lib_id "ABX00042:ABX00042") (at 76.2 76.2 0) (unit 1)
     (in_bom yes) (on_board yes) (dnp no) (fields_autoplaced)
     (property "Reference" "U1" (at 76.2 21.59 0)

Commit message: Finished routing
Parts:
- J1: footprint Connector_PinHeader_1.27mm:PinHeader_2x07_P1.27mm_Vertical_SMD -> STDC14_header:PinHeader_2x07_P1.27mm_Vertical_SMD
- U1: value ABX00042 -> DF40HC(3.5)-80DS-0.4V(51); footprint Portenta:MODULE_ABX00042 -> Portenta:MODULE_ABX00042_NOSCREWS
Connections:
- net +3.3V: now also U1.J1_72 (V-SDCARD)
- net +5V: now reaches U1.J1_23 (USB1_VBUS)
- net SDC_CD: now reaches U1.J1_38 (UART0_RTS)
- net SDC_CLK: now reaches U1.J1_55 (SDC_CLK)
- net SDC_CMD: now reaches U1.J1_57 (SDC_CMD)
- net SDC_D0: now reaches U1.J1_59 (SDC_D0)
- net SDC_D1: now reaches U1.J1_61 (SDC_D1)
- net SDC_D2: now reaches U1.J1_63 (SDC_D2)
- net SDC_D3: now reaches U1.J1_65 (SDC_D3)
- net RADAR_RST renamed RADAR_nRST
- no-connect marks 68 -> 59
Other:
- note added: "Active high!"
- note added: "BOOT0"
- note added: "Bus shared with PMIC, crypto, video"
- note added: "DSI only pins"
- note added: "From Portenta H7 schematic:"
- note added: "PA0_C"
- note added: "PA10"
- note added: "PA11"
- note added: "PA12"
- note added: "PA13"
- note added: "PA14"
- note added: "PA1_C"
- note added: "PA8"
- note added: "PA9"
- note added: "PB14"
- note added: "PB15"
- note added: "PB2"
- note added: "PB3"
- note added: "PB4"
- note added: "PB8"
- note added: "PC13"
- note added: "PC15"
- note added: "PC2_C"
- note added: "PC3_C"
- note added: "PC6"
- note added: "PC7"
- note added: "PD4"
- note added: "PD5"
- note added: "PD6"
- note added: "PD7"
- note added: "PE2"
- note added: "PE3"
- note added: "PG10"
- note added: "PG3"
- note added: "PG7"
- note added: "PH13"
- note added: "PH15"
- note added: "PH6"
- note added: "PI10"
- note added: "PI13"
- note added: "PI3"
- note added: "PI8"
- note added: "PJ10"
- note added: "PJ11"
- note added: "PJ7"
- note added: "PJ8"
- note added: "PJ9"
- note added: "PK1"
- note added: "PMIC pins"
- note added: "Pins shared with camera"
- note added: "Pins shared with radar"
- note added: "Portenta onboard USB"
- note added: "RX"
- note added: "SWO pin shared with SD D2!"
- note added: "TX"
- note added: "USB for console"
- note added: "microSD"
- note removed: "Shared with PMIC, crypto"

Commit message: Add testpoints, 0ohm, led, logos
Parts:
- added D1: Würth 150066M153000, 150066M153000:Würth_150066M153000, symbol Device:LED_RGBA
- added R25: 1k, Resistor_SMD:R_0603_1608Metric, symbol Device:R
- added R26: 470, Resistor_SMD:R_0603_1608Metric, symbol Device:R
- added R27: 220, Resistor_SMD:R_0603_1608Metric, symbol Device:R
Connections:
- net +3.3V: now also D1.4 (A)
- net nLEDR: now reaches U1.J2_63 (PWM_3)
- net nLEDR: now also R25.1
- net nLEDG: now reaches U1.J2_65 (PWM_4)
- net nLEDG: now also R26.1
- net nLEDB: now reaches U1.J2_67 (PWM_5)
- net nLEDB: now also R27.1
- new net CATB: D1.3 (BK), R27.2
- new net CATG: D1.2 (GK), R26.2
- new net CATR: D1.1 (RK), R25.2
- no-connect marks 59 -> 56
Other:
- note added: "Calculated for 20mcd"
Changed lines of the file:
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@@
   (title_block
     (title "Heterogeneous radar, RGB, and ToF sensor board")
-    (date "2023-04-24")
-    (rev "1.2")
+    (date "2023-04-25")
+    (rev "1.3")
     (company "Center for Project-Based Learning")
     (comment 1 "Zoltán Marcsek")
@@
   )
   (no_connect (at 190.5 81.28))
-  (no_connect (at 241.3 96.52))
   (no_connect (at 88.9 165.1))
   (no_connect (at 101.6 43.18))
@@
   (no_connect (at 190.5 66.04))
   (no_connect (at 101.6 50.8))
-  (no_connect (at 241.3 99.06))
   (no_connect (at 190.5 83.82))
   (no_connect (at 50.8 58.42))
   (no_connect (at 101.6 45.72))
-  (no_connect (at 241.3 93.98))
   (no_connect (at 50.8 91.44))
   (no_connect (at 101.6 109.22))
@@
     (stroke (width 0) (type default))
   )
+  (wire (pts (xy 256.54 93.98) (xy 241.3 93.98))
+    (stroke (width 0) (type default))
+  )
   (polyline (pts (xy 129.54 71.755) (xy 132.08 71.755))
     (stroke (width 0) (type default))
@@
     (stroke (width 0) (type default))
   )
+  (wire (pts (xy 251.46 99.06) (xy 251.46 132.08))
+    (stroke (width 0) (type default))
+  )
   (bus (pts (xy 38.1 38.1) (xy 38.1 40.64))
     (stroke (width 0) (type default))
@@
     (stroke (width 0) (type default))
   )
+  (wire (pts (xy 264.16 121.92) (xy 267.97 121.92))
+    (stroke (width 0) (type default))
+  )
   (polyline (pts (xy 129.54 102.235) (xy 132.08 102.235))
     (stroke (width 0) (type default))
@@
     (stroke (width 0) (type default))
   )
+  (wire (pts (xy 264.16 127) (xy 267.97 127))
+    (stroke (width 0) (type default))
+  )
   (bus (pts (xy 255.27 73.66) (xy 254 73.66))
     (stroke (width 0) (type default))
@@
     (stroke (width 0) (type default))
   )
+  (wire (pts (xy 264.16 132.08) (xy 267.97 132.08))
+    (stroke (width 0) (type default))
+  )
   (polyline (pts (xy 190.5 95.25) (xy 189.23 95.25))
     (stroke (width 0) (type default))
@@
     (stroke (width 0) (type default))
   )
+  (wire (pts (xy 241.3 99.06) (xy 251.46 99.06))
+    (stroke (width 0) (type default))
+  )
   (polyline (pts (xy 190.5 41.91) (xy 189.23 41.91))
     (stroke (width 0) (type default))
@@
   )
   (wire (pts (xy 40.64 81.28) (xy 50.8 81.28))
+    (stroke (width 0) (type default))
+  )
+  (wire (pts (xy 279.4 127) (xy 278.13 127))
     (stroke (width 0) (type default))
   )
@@
     (stroke (width 0) (type default))
   )
+  (wire (pts (xy 254 96.52) (xy 254 127))
+    (stroke (width 0) (type default))
+  )
   (polyline (pts (xy 22.86 94.615) (xy 20.32 94.615))
     (stroke (width 0) (type default))
@@
     (stroke (width 0) (type default))
   )
+  (wire (pts (xy 241.3 96.52) (xy 254 96.52))
+    (stroke (width 0) (type default))
+  )
   (wire (pts (xy 104.14 124.46) (xy 101.6 124.46))
     (stroke (width 0) (type default))
@@
     (stroke (width 0) (type default))
   )
+  (wire (pts (xy 251.46 132.08) (xy 256.54 132.08))
+    (stroke (width 0) (type default))
+  )
   (bus (pts (xy 38.1 99.06) (xy 38.1 101.6))
     (stroke (width 0) (type default))
@@
   )
   (polyline (pts (xy 269.24 84.455) (xy 271.78 84.455))
+    (stroke (width 0) (type default))
+  )
+  (wire (pts (xy 256.54 121.92) (xy 256.54 93.98))
     (stroke (width 0) (type default))
   )
@@
     (stroke (width 0) (type default))
   )
+  (wire (pts (xy 254 127) (xy 256.54 127))
+    (stroke (width 0) (type default))
+  )
   (wire (pts (xy 241.3 63.5) (xy 254 63.5))
     (stroke (width 0) (type default))
@@
   )
   (bus (pts (xy 38.1 45.72) (xy 38.1 48.26))
+    (stroke (width 0) (type default))
+  )
+  (wire (pts (xy 279.4 125.73) (xy 279.4 127))
     (stroke (width 0) (type default))
   )
@@
     (effects (font (face "Asap") (size 2 2)) (justify left bottom))
   )
+  (text "Calculated for 20mcd" (at 259.08 138.43 0)
+    (effects (font (size 1.27 1.27)) (justify left bottom))
+  )
   (text "PC15" (at 171.45 106.68 0)
     (effects (font (size 1.27 1.27)) (justify left bottom))
@@
     (effects (font (size 1.27 1.27)) (justify right bottom))
   )
+  (label "nLEDR" (at 241.3 93.98 0) (fields_autoplaced)
+    (effects (font (size 1.27 1.27)) (justify left bottom))
+  )
   (label "ETH_A+" (at 50.8 38.1 180) (fields_autoplaced)
     (effects (font (size 1.27 1.27)) (justify right bottom))
@@
     (effects (font (size 1.27 1.27)) (justify left bottom))
   )
+  (label "CATG" (at 264.16 127 0) (fields_autoplaced)
+    (effects (font (size 1.27 1.27)) (justify left bottom))
+  )
   (label "ETH_LED2" (at 50.8 50.8 180) (fields_autoplaced)
     (effects (font (size 1.27 1.27)) (justify right bottom))
   )
+  (label "CATB" (at 264.16 132.08 0) (fields_autoplaced)
+    (effects (font (size 1.27 1.27)) (justify left bottom))
+  )
   (label "CAM_D5" (at 241.3 43.18 0) (fields_autoplaced)
     (effects (font (size 1.27 1.27)) (justify left bottom))
@@
     (effects (font (size 1.27 1.27)) (justify right bottom))
   )
+  (label "nLEDB" (at 241.3 99.06 0) (fields_autoplaced)
+    (effects (font (size 1.27 1.27)) (justify left bottom))
+  )
   (label "UART4_RX" (at 114.3 71.12 180) (fields_autoplaced)
     (effects (font (size 1.27 1.27)) (justify right bottom))
@@
     (effects (font (size 1.27 1.27)) (justify left bottom))
   )
+  (label "nLEDG" (at 241.3 96.52 0) (fields_autoplaced)
+    (effects (font (size 1.27 1.27)) (justify left bottom))
+  )
   (label "SPI2_SCK" (at 241.3 78.74 0) (fields_autoplaced)
     (effects (font (size 1.27 1.27)) (justify left bottom))
   )
   (label "nRST" (at 38.1 114.3 0) (fields_autoplaced)
+    (effects (font (size 1.27 1.27)) (justify left bottom))
+  )
+  (label "CATR" (at 264.16 121.92 0) (fields_autoplaced)
     (effects (font (size 1.27 1.27)) (justify left bottom))
   )
@@
     )
   )
+  (symbol (lib_id "power:+3.3V") (at 279.4 125.73 0) (unit 1)
+    (in_bom yes) (on_board yes) (dnp no) (fields_autoplaced)
+    (property "Reference" "#PWR0108" (at 279.4 129.54 0)
+      (effects (font (size 1.27 1.27)) hide)
+    )
+    (property "Value" "+3.3V" (at 279.4 121.92 0)
+      (effects (font (size 1.27 1.27)))
+    )
+    (property "Footprint" "" (at 279.4 125.73 0)
+      (effects (font (size 1.27 1.27)) hide)
+    )
+    (property "Datasheet" "" (at 279.4 125.73 0)
+      (effects (font (size 1.27 1.27)) hide)
+    )
+    (pin "1")
+    (instances
+      (project "radartof-hardware"
+        (path "/03db8980-0fb1-4523-a968-8d3a1d96010b/87bd9a1d-ab0d-4743-af65-7117412c655d"
+          (reference "#PWR0108") (unit 1)
+        )
+      )
+    )
+  )
   (symbol (lib_id "power:+3.3V") (at 104.14 27.94 0) (unit 1)
     (in_bom yes) (on_board yes) (dnp no) (fields_autoplaced)
@@
         (path "/03db8980-0fb1-4523-a968-8d3a1d96010b/87bd9a1d-ab0d-4743-af65-7117412c655d"
           (reference "#PWR02") (unit 1)
+        )
+      )
+    )
+  )
+  (symbol (lib_id "Device:R") (at 260.35 132.08 90) (unit 1)
+    (in_bom yes) (on_board yes) (dnp no)
+    (property "Reference" "R27" (at 260.35 129.54 90)
+      (effects (font (size 1.27 1.27)))
+    )
+    (property "Value" "220" (at 260.35 132.08 90)
+      (effects (font (size 1.27 1.27)))
+    )
+    (property "Footprint" "Resistor_SMD:R_0603_1608Metric" (at 260.35 133.858 90)
+      (effects (font (size 1.27 1.27)) hide)
+    )
+    (property "Datasheet" "~" (at 260.35 132.08 0)
+      (effects (font (size 1.27 1.27)) hide)
+    )
+    (pin "1")
+    (pin "2")
+    (instances
+      (project "radartof-hardware"
+        (path "/03db8980-0fb1-4523-a968-8d3a1d96010b/87bd9a1d-ab0d-4743-af65-7117412c655d"
+          (reference "R27") (unit 1)
         )
       )
@@
         )
       )
+    )
+  )
+  (symbol (lib_id "Device:R") (at 260.35 121.92 90) (unit 1)
+    (in_bom yes) (on_board yes) (dnp no)
+    (property "Reference" "R25" (at 260.35 119.38 90)
+      (effects (font (size 1.27 1.27)))
+    )
+    (property "Value" "1k" (at 260.35 121.92 90)
+      (effects (font (size 1.27 1.27)))
+    )
+    (property "Footprint" "Resistor_SMD:R_0603_1608Metric" (at 260.35 123.698 90)
+      (effects (font (size 1.27 1.27)) hide)
+    )
+    (property "Datasheet" "~" (at 260.35 121.92 0)
+      (effects (font (size 1.27 1.27)) hide)
+    )
+    (pin "1")
+    (pin "2")
+    (instances
+      (project "radartof-hardware"
+        (path "/03db8980-0fb1-4523-a968-8d3a1d96010b/87bd9a1d-ab0d-4743-af65-7117412c655d"
+          (reference "R25") (unit 1)
+        )
+      )
+    )
+  )
+  (symbol (lib_id "Device:R") (at 260.35 127 90) (unit 1)
+    (in_bom yes) (on_board yes) (dnp no)
+    (property "Reference" "R26" (at 260.35 124.46 90)
+      (effects (font (size 1.27 1.27)))
+    )
+    (property "Value" "470" (at 260.35 127 90)
+      (effects (font (size 1.27 1.27)))
+    )
+    (property "Footprint" "Resistor_SMD:R_0603_1608Metric" (at 260.35 128.778 90)
+      (effects (font (size 1.27 1.27)) hide)
+    )
+    (property "Datasheet" "~" (at 260.35 127 0)
+      (effects (font (size 1.27 1.27)) hide)
+    )
+    (pin "1")
+    (pin "2")
+    (instances
+      (project "radartof-hardware"
+        (path "/03db8980-0fb1-4523-a968-8d3a1d96010b/87bd9a1d-ab0d-4743-af65-7117412c655d"
+          (reference "R26") (unit 1)
+        )
+      )
+    )
+  )
+  (symbol (lib_id "Device:LED_RGBA") (at 273.05 127 0) (unit 1)
+    (in_bom yes) (on_board yes) (dnp no) (fields_autoplaced)
+    (property "Reference" "D1" (at 273.05 114.3 0)
+      (effects (font (size 1.27 1.27)))
+    )
+    (property "Value" "Würth 150066M153000" (at 273.05 116.84 0)
+      (effects (font (size 1.27 1.27)))
+    )
+    (property "Footprint" "150066M153000:Würth_150066M153000" (at 273.05 128.27 0)
+      (effects (font (size 1.27 1.27)) hide)
+    )
+    (property "Datasheet" "~" (at 273.05 128.27 0)
+      (effects (font (size 1.27 1.27)) hide)
+    )
+    (pin "1")
+    (pin "2")
+    (pin "3")
+    (pin "4")
+    (instances
+      (project "radartof-hardware"
+        (path "/03db8980-0fb1-4523-a968-8d3a1d96010b/87bd9a1d-ab0d-4743-af65-7117412c655d"
+          (reference "D1") (unit 1)
+        )
+      )
