File: hardware/mcu.kicad_sch (KiCad schematic)
At the start: 6 parts, among them J1 Debug, U1 DF40HC(3.5)-80DS-0.4V(51)

Commit message: Final fixes, manufacturing
Parts:
- D1: MANUFACTURER (none) -> Wuerth; MOUSER NO (none) -> 710-150066M153000; PART NO (none) -> 150066M153000
- J1: MANUFACTURER (none) -> Samtec; MOUSER NO (none) -> 200-FTSH10701LDVKPTR; PART NO (none) -> FTSH-107-01-L-DV-K-P-TR
- R25: MANUFACTURER (none) -> Vishay / Dale; MOUSER NO (none) -> 71-CRCW06031K00FKEAC; PART NO (none) -> CRCW06031K00FKEAC
- R26: MANUFACTURER (none) -> Vishay / Dale; MOUSER NO (none) -> 71-CRCW0603470RFKEAC; PART NO (none) -> CRCW0603470RFKEAC
- R27: MANUFACTURER (none) -> Vishay / Dale; MOUSER NO (none) -> 71-CRCW0603220RFKEAC; PART NO (none) -> CRCW0603220RFKEAC
- U1: MANUFACTURER Arduino -> Hirose; MOUSER NO (none) -> 798-DF40HC3580DS4V51; PART NO (none) -> DF40HC(3.5)-80DS-0.4V(51)
Changed lines of the file:
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@@
   (title_block
     (title "Heterogeneous radar, RGB, and ToF sensor board")
-    (date "2023-04-25")
-    (rev "1.3")
+    (date "2023-04-26")
+    (rev "1.4")
     (company "Center for Project-Based Learning")
     (comment 1 "Zoltán Marcsek")
@@
       (effects (font (size 1.27 1.27)) hide)
     )
+    (property "MOUSER NO" "200-FTSH10701LDVKPTR" (at 76.2 165.1 0)
+      (effects (font (size 1.27 1.27)) hide)
+    )
+    (property "PART NO" "FTSH-107-01-L-DV-K-P-TR" (at 76.2 165.1 0)
+      (effects (font (size 1.27 1.27)) hide)
+    )
+    (property "MANUFACTURER" "Samtec" (at 76.2 165.1 0)
+      (effects (font (size 1.27 1.27)) hide)
+    )
     (pin "1")
     (pin "10")
@@
       (effects (font (size 1.27 1.27)) hide)
     )
-    (property "Datasheet" "~" (at 260.35 132.08 0)
+    (property "Datasheet" "https://www.mouser.ch/datasheet/2/427/crcwce3-1762584.pdf" (at 260.35 132.08 0)
+      (effects (font (size 1.27 1.27)) hide)
+    )
+    (property "MOUSER NO" "71-CRCW0603220RFKEAC" (at 260.35 132.08 0)
+      (effects (font (size 1.27 1.27)) hide)
+    )
+    (property "PART NO" "CRCW0603220RFKEAC" (at 260.35 132.08 0)
+      (effects (font (size 1.27 1.27)) hide)
+    )
+    (property "MANUFACTURER" "Vishay / Dale" (at 260.35 132.08 0)
       (effects (font (size 1.27 1.27)) hide)
     )
@@
       (effects (font (size 1.27 1.27)) (justify bottom) hide)
     )
-    (property "Datasheet" "" (at 215.9 76.2 0)
+    (property "Datasheet" "https://www.hirose.com/en/product/document?clcode=CL0684-4162-7-51&productname=DF40HC(3.5)-80DS-0.4V(51)&series=DF40&documenttype=2DDrawing&lang=en&documentid=0001142901" (at 215.9 76.2 0)
       (effects (font (size 1.27 1.27)) hide)
     )
@@
       (effects (font (size 1.27 1.27)) (justify bottom) hide)
     )
-    (property "MANUFACTURER" "Arduino" (at 215.9 76.2 0)
+    (property "MANUFACTURER" "Hirose" (at 215.9 76.2 0)
       (effects (font (size 1.27 1.27)) (justify bottom) hide)
+    )
+    (property "MOUSER NO" "798-DF40HC3580DS4V51" (at 215.9 76.2 0)
+      (effects (font (size 1.27 1.27)) hide)
+    )
+    (property "PART NO" "DF40HC(3.5)-80DS-0.4V(51)" (at 215.9 76.2 0)
+      (effects (font (size 1.27 1.27)) hide)
     )
     (pin "J1_1")
@@
       (effects (font (size 1.27 1.27)) hide)
     )
-    (property "Datasheet" "~" (at 260.35 121.92 0)
+    (property "Datasheet" "https://www.mouser.ch/datasheet/2/427/crcwce3-1762584.pdf" (at 260.35 121.92 0)
+      (effects (font (size 1.27 1.27)) hide)
+    )
+    (property "MOUSER NO" "71-CRCW06031K00FKEAC" (at 260.35 121.92 0)
+      (effects (font (size 1.27 1.27)) hide)
+    )
+    (property "PART NO" "CRCW06031K00FKEAC" (at 260.35 121.92 0)
+      (effects (font (size 1.27 1.27)) hide)
+    )
+    (property "MANUFACTURER" "Vishay / Dale" (at 260.35 121.92 0)
       (effects (font (size 1.27 1.27)) hide)
     )
@@
       (effects (font (size 1.27 1.27)) hide)
     )
-    (property "Datasheet" "~" (at 260.35 127 0)
+    (property "Datasheet" "https://www.mouser.ch/datasheet/2/427/crcwce3-1762584.pdf" (at 260.35 127 0)
+      (effects (font (size 1.27 1.27)) hide)
+    )
+    (property "MOUSER NO" "71-CRCW0603470RFKEAC" (at 260.35 127 0)
+      (effects (font (size 1.27 1.27)) hide)
+    )
+    (property "PART NO" "CRCW0603470RFKEAC" (at 260.35 127 0)
+      (effects (font (size 1.27 1.27)) hide)
+    )
+    (property "MANUFACTURER" "Vishay / Dale" (at 260.35 127 0)
       (effects (font (size 1.27 1.27)) hide)
     )
@@
       (effects (font (size 1.27 1.27)) hide)
     )
-    (property "Datasheet" "~" (at 273.05 128.27 0)
+    (property "Datasheet" "https://www.we-online.com/components/products/datasheet/150066M153000.pdf" (at 273.05 128.27 0)
+      (effects (font (size 1.27 1.27)) hide)
+    )
+    (property "MOUSER NO" "710-150066M153000" (at 273.05 127 0)
+      (effects (font (size 1.27 1.27)) hide)
+    )
+    (property "PART NO" "150066M153000" (at 273.05 127 0)
+      (effects (font (size 1.27 1.27)) hide)
+    )
+    (property "MANUFACTURER" "Wuerth" (at 273.05 127 0)
       (effects (font (size 1.27 1.27)) hide)
     )
@@
       (effects (font (size 1.27 1.27)) (justify bottom) hide)
     )
-    (property "Datasheet" "" (at 76.2 76.2 0)
+    (property "Datasheet" "https://www.hirose.com/en/product/document?clcode=CL0684-4162-7-51&productname=DF40HC(3.5)-80DS-0.4V(51)&series=DF40&documenttype=2DDrawing&lang=en&documentid=0001142901" (at 76.2 76.2 0)
       (effects (font (size 1.27 1.27)) hide)
     )
@@
       (effects (font (size 1.27 1.27)) (justify bottom) hide)
     )
-    (property "MANUFACTURER" "Arduino" (at 76.2 76.2 0)
+    (property "MANUFACTURER" "Hirose" (at 76.2 76.2 0)
       (effects (font (size 1.27 1.27)) (justify bottom) hide)
     )
+    (property "MOUSER NO" "798-DF40HC3580DS4V51" (at 76.2 76.2 0)
+      (effects (font (size 1.27 1.27)) hide)
+    )
+    (property "PART NO" "DF40HC(3.5)-80DS-0.4V(51)" (at 76.2 76.2 0)
+      (effects (font (size 1.27 1.27)) hide)
+    )
     (pin "J1_1")
