File: hardware/microsd.kicad_sch (KiCad schematic)
At the start: 3 parts, among them J3 1140084168

Commit message: Add testpoints, 0ohm, led, logos
Parts:
- added R21: 0, Resistor_SMD:R_0603_1608Metric, symbol Device:R
Connections:
- net SDC_D2: now also R21.1; no longer J3.1 (DAT2)
- new net: J3.1 (DAT2), R21.2
Changed lines of the file:
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@@
   (title_block
     (title "Heterogeneous radar, RGB, and ToF sensor board")
-    (date "2023-04-24")
-    (rev "1.2")
+    (date "2023-04-25")
+    (rev "1.3")
     (company "Center for Project-Based Learning")
     (comment 1 "Zoltán Marcsek")
@@
   (junction (at 177.8 97.79) (diameter 0) (color 0 0 0 0)
   )
-  (bus_entry (at 88.9 91.44) (size 2.54 2.54)
-    (stroke (width 0) (type default))
-  )
-  (bus_entry (at 88.9 99.06) (size 2.54 2.54)
-    (stroke (width 0) (type default))
-  )
-  (bus_entry (at 88.9 104.14) (size 2.54 2.54)
-    (stroke (width 0) (type default))
-  )
-  (bus_entry (at 88.9 111.76) (size 2.54 2.54)
-    (stroke (width 0) (type default))
-  )
-  (bus_entry (at 88.9 93.98) (size 2.54 2.54)
-    (stroke (width 0) (type default))
-  )
-  (bus_entry (at 88.9 88.9) (size 2.54 2.54)
-    (stroke (width 0) (type default))
-  )
-  (bus_entry (at 88.9 106.68) (size 2.54 2.54)
-    (stroke (width 0) (type default))
-  )
-  (bus (pts (xy 88.9 91.44) (xy 88.9 93.98))
-    (stroke (width 0) (type default))
-  )
-  (wire (pts (xy 91.44 91.44) (xy 116.84 91.44))
-    (stroke (width 0) (type default))
-  )
-  (bus (pts (xy 88.9 106.68) (xy 88.9 111.76))
+  (bus_entry (at 76.2 91.44) (size 2.54 2.54)
+    (stroke (width 0) (type default))
+  )
+  (bus_entry (at 76.2 99.06) (size 2.54 2.54)
+    (stroke (width 0) (type default))
+  )
+  (bus_entry (at 76.2 104.14) (size 2.54 2.54)
+    (stroke (width 0) (type default))
+  )
+  (bus_entry (at 76.2 111.76) (size 2.54 2.54)
+    (stroke (width 0) (type default))
+  )
+  (bus_entry (at 76.2 93.98) (size 2.54 2.54)
+    (stroke (width 0) (type default))
+  )
+  (bus_entry (at 76.2 88.9) (size 2.54 2.54)
+    (stroke (width 0) (type default))
+  )
+  (bus_entry (at 76.2 106.68) (size 2.54 2.54)
+    (stroke (width 0) (type default))
+  )
+  (wire (pts (xy 78.74 93.98) (xy 116.84 93.98))
+    (stroke (width 0) (type default))
+  )
+  (bus (pts (xy 76.2 91.44) (xy 76.2 93.98))
+    (stroke (width 0) (type default))
+  )
+  (bus (pts (xy 76.2 106.68) (xy 76.2 111.76))
     (stroke (width 0) (type default))
   )
@@
     (stroke (width 0) (type default))
   )
-  (bus (pts (xy 88.9 88.9) (xy 88.9 91.44))
-    (stroke (width 0) (type default))
-  )
-  (wire (pts (xy 91.44 106.68) (xy 116.84 106.68))
-    (stroke (width 0) (type default))
-  )
-  (bus (pts (xy 88.9 104.14) (xy 88.9 106.68))
+  (bus (pts (xy 76.2 88.9) (xy 76.2 91.44))
+    (stroke (width 0) (type default))
+  )
+  (bus (pts (xy 76.2 104.14) (xy 76.2 106.68))
+    (stroke (width 0) (type default))
+  )
+  (wire (pts (xy 78.74 106.68) (xy 116.84 106.68))
     (stroke (width 0) (type default))
   )
@@
     (stroke (width 0) (type default))
   )
-  (bus (pts (xy 88.9 93.98) (xy 88.9 99.06))
-    (stroke (width 0) (type default))
-  )
-  (wire (pts (xy 91.44 109.22) (xy 116.84 109.22))
+  (bus (pts (xy 76.2 93.98) (xy 76.2 99.06))
+    (stroke (width 0) (type default))
+  )
+  (wire (pts (xy 105.41 91.44) (xy 116.84 91.44))
+    (stroke (width 0) (type default))
+  )
+  (wire (pts (xy 78.74 109.22) (xy 116.84 109.22))
     (stroke (width 0) (type default))
   )
@@
     (stroke (width 0) (type default))
   )
+  (wire (pts (xy 78.74 96.52) (xy 116.84 96.52))
+    (stroke (width 0) (type default))
+  )
+  (wire (pts (xy 78.74 91.44) (xy 97.79 91.44))
+    (stroke (width 0) (type default))
+  )
   (wire (pts (xy 114.3 111.76) (xy 114.3 116.84))
     (stroke (width 0) (type default))
   )
-  (wire (pts (xy 91.44 101.6) (xy 116.84 101.6))
-    (stroke (width 0) (type default))
-  )
-  (wire (pts (xy 91.44 93.98) (xy 116.84 93.98))
-    (stroke (width 0) (type default))
-  )
-  (bus (pts (xy 88.9 99.06) (xy 88.9 104.14))
+  (wire (pts (xy 78.74 101.6) (xy 116.84 101.6))
+    (stroke (width 0) (type default))
+  )
+  (bus (pts (xy 76.2 99.06) (xy 76.2 104.14))
     (stroke (width 0) (type default))
   )
@@
     (stroke (width 0) (type default))
   )
-  (bus (pts (xy 88.9 76.2) (xy 88.9 88.9))
-    (stroke (width 0) (type default))
-  )
-  (wire (pts (xy 91.44 114.3) (xy 116.84 114.3))
+  (bus (pts (xy 76.2 76.2) (xy 76.2 88.9))
+    (stroke (width 0) (type default))
+  )
+  (wire (pts (xy 78.74 114.3) (xy 116.84 114.3))
     (stroke (width 0) (type default))
   )
@@
     (stroke (width 0) (type default))
   )
-  (wire (pts (xy 91.44 96.52) (xy 116.84 96.52))
-    (stroke (width 0) (type default))
-  )
   (wire (pts (xy 177.8 105.41) (xy 190.5 105.41))
     (stroke (width 0) (type default))
   )
-  (label "SDC_CLK" (at 101.6 101.6 0) (fields_autoplaced)
-    (effects (font (size 1.27 1.27)) (justify left bottom))
-  )
-  (label "SDC_CMD" (at 101.6 96.52 0) (fields_autoplaced)
-    (effects (font (size 1.27 1.27)) (justify left bottom))
-  )
-  (label "SDC_D2" (at 101.6 91.44 0) (fields_autoplaced)
-    (effects (font (size 1.27 1.27)) (justify left bottom))
-  )
-  (label "SDC_D1" (at 101.6 109.22 0) (fields_autoplaced)
-    (effects (font (size 1.27 1.27)) (justify left bottom))
-  )
-  (label "SDC_D0" (at 101.6 106.68 0) (fields_autoplaced)
-    (effects (font (size 1.27 1.27)) (justify left bottom))
-  )
-  (label "SDC_D3" (at 101.6 93.98 0) (fields_autoplaced)
-    (effects (font (size 1.27 1.27)) (justify left bottom))
-  )
-  (label "SDC_CD" (at 101.6 114.3 0) (fields_autoplaced)
-    (effects (font (size 1.27 1.27)) (justify left bottom))
-  )
-  (hierarchical_label "{SDC}" (shape bidirectional) (at 88.9 76.2 90) (fields_autoplaced)
+  (label "SDC_CLK" (at 88.9 101.6 0) (fields_autoplaced)
+    (effects (font (size 1.27 1.27)) (justify left bottom))
+  )
+  (label "SDC_CMD" (at 88.9 96.52 0) (fields_autoplaced)
+    (effects (font (size 1.27 1.27)) (justify left bottom))
+  )
+  (label "SDC_D2" (at 88.9 91.44 0) (fields_autoplaced)
+    (effects (font (size 1.27 1.27)) (justify left bottom))
+  )
+  (label "SDC_D1" (at 88.9 109.22 0) (fields_autoplaced)
+    (effects (font (size 1.27 1.27)) (justify left bottom))
+  )
+  (label "SDC_D0" (at 88.9 106.68 0) (fields_autoplaced)
+    (effects (font (size 1.27 1.27)) (justify left bottom))
+  )
+  (label "SDC_D3" (at 88.9 93.98 0) (fields_autoplaced)
+    (effects (font (size 1.27 1.27)) (justify left bottom))
+  )
+  (label "SDC_CD" (at 88.9 114.3 0) (fields_autoplaced)
+    (effects (font (size 1.27 1.27)) (justify left bottom))
+  )
+  (hierarchical_label "{SDC}" (shape bidirectional) (at 76.2 76.2 90) (fields_autoplaced)
     (effects (font (size 1.27 1.27)) (justify left))
   )
@@
         )
       )
+    )
+  )
+  (symbol (lib_id "Device:R") (at 101.6 91.44 90) (unit 1)
+    (in_bom yes) (on_board yes) (dnp no)
+    (property "Reference" "R21" (at 101.6 88.9 90)
+      (effects (font (size 1.27 1.27)))
+    )
+    (property "Value" "0" (at 101.6 91.44 90)
+      (effects (font (size 1.27 1.27)))
+    )
+    (property "Footprint" "Resistor_SMD:R_0603_1608Metric" (at 101.6 93.218 90)
+      (effects (font (size 1.27 1.27)) hide)
+    )
+    (property "Datasheet" "~" (at 101.6 91.44 0)
+      (effects (font (size 1.27 1.27)) hide)
+    )
+    (pin "1")
+    (pin "2")
+    (instances
+      (project "radartof-hardware"
+        (path "/03db8980-0fb1-4523-a968-8d3a1d96010b/1c3d9fbe-6cf2-4d26-9b7d-c2f580c91270"
+          (reference "R21") (unit 1)
+        )
+      )

Commit message: Final fixes, manufacturing
Parts:
- C49: MANUFACTURER (none) -> KEMET; MOUSER NO (none) -> 80-C603C104K5RAC3121; PART NO (none) -> C0603C104K5RAC3121
- C50: MANUFACTURER (none) -> Murata; MOUSER NO (none) -> 81-GRM188Z71A106KA3D; PART NO (none) -> GRM188Z71A106KA73D
- J3: MANUFACTURER (none) -> Amphenol CS; MOUSER NO (none) -> 523-114-00841-68; PART NO (none) -> 1140084168
- R21: MANUFACTURER (none) -> Vishay / Dale; MOUSER NO (none) -> 71-CRCW06030000Z0EBC; PART NO (none) -> CRCW06030000Z0EBC
Changed lines of the file:
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@@
   (title_block
     (title "Heterogeneous radar, RGB, and ToF sensor board")
-    (date "2023-04-25")
-    (rev "1.3")
+    (date "2023-04-26")
+    (rev "1.4")
     (company "Center for Project-Based Learning")
     (comment 1 "Zoltán Marcsek")
@@
       (effects (font (size 1.27 1.27)) hide)
     )
-    (property "Datasheet" "~" (at 190.5 101.6 0)
+    (property "Datasheet" "https://www.mouser.ch/datasheet/2/281/1/GRM188Z71A106KA73_01A-1986029.pdf" (at 190.5 101.6 0)
+      (effects (font (size 1.27 1.27)) hide)
+    )
+    (property "MANUFACTURER" "Murata" (at 190.5 101.6 0)
+      (effects (font (size 1.27 1.27)) hide)
+    )
+    (property "MOUSER NO" "81-GRM188Z71A106KA3D" (at 190.5 101.6 0)
+      (effects (font (size 1.27 1.27)) hide)
+    )
+    (property "PART NO" "GRM188Z71A106KA73D" (at 190.5 101.6 0)
       (effects (font (size 1.27 1.27)) hide)
     )
@@
       (effects (font (size 1.27 1.27)) hide)
     )
-    (property "Datasheet" "~" (at 101.6 91.44 0)
+    (property "Datasheet" "https://www.mouser.ch/datasheet/2/427/crcwce3-1762584.pdf" (at 101.6 91.44 0)
+      (effects (font (size 1.27 1.27)) hide)
+    )
+    (property "MOUSER NO" "71-CRCW06030000Z0EBC" (at 101.6 91.44 0)
+      (effects (font (size 1.27 1.27)) hide)
+    )
+    (property "PART NO" "CRCW06030000Z0EBC" (at 101.6 91.44 0)
+      (effects (font (size 1.27 1.27)) hide)
+    )
+    (property "MANUFACTURER" "Vishay / Dale" (at 101.6 91.44 0)
       (effects (font (size 1.27 1.27)) hide)
     )
@@
       (effects (font (size 1.27 1.27)) hide)
     )
-    (property "Datasheet" "~" (at 177.8 101.6 0)
+    (property "Datasheet" "https://www.mouser.ch/datasheet/2/212/KEM_C1023_X7R_AUTO_SMD-1093309.pdf" (at 177.8 101.6 0)
+      (effects (font (size 1.27 1.27)) hide)
+    )
+    (property "MANUFACTURER" "KEMET" (at 177.8 101.6 0)
+      (effects (font (size 1.27 1.27)) hide)
+    )
+    (property "MOUSER NO" "80-C603C104K5RAC3121" (at 177.8 101.6 0)
+      (effects (font (size 1.27 1.27)) hide)
+    )
+    (property "PART NO" "C0603C104K5RAC3121" (at 177.8 101.6 0)
       (effects (font (size 1.27 1.27)) hide)
     )
@@
       (effects (font (size 1.27 1.27)) hide)
     )
+    (property "MOUSER NO" "523-114-00841-68" (at 139.7 101.6 0)
+      (effects (font (size 1.27 1.27)) hide)
+    )
+    (property "PART NO" "1140084168" (at 139.7 101.6 0)
+      (effects (font (size 1.27 1.27)) hide)
+    )
+    (property "MANUFACTURER" "Amphenol CS" (at 139.7 101.6 0)
+      (effects (font (size 1.27 1.27)) hide)
+    )
