File: hardware/radar.kicad_sch (KiCad schematic)
At the start: 5 parts, among them U4 TLV74318 SOT23-5, X1 OSC-80MHz

Commit message: final-ish schematic
Parts:
- removed U4: TLV74318 SOT23-5, Package_TO_SOT_SMD:SOT-23-5, symbol Regulator_Linear:TLV70012_SOT23-5
- removed X1: OSC-80MHz, Oscillator:Oscillator_SMD_ECS_2520MV-xxx-xx-4Pin_2.5x2.0mm, symbol Oscillator:ECS-2520MV-xxx-xx
- added C15, C20, C24, C26, C27, C29: 10u, Capacitor_SMD:C_0603_1608Metric, symbol Device:C
- added C21, C30, C32, C33, C36, C38, C40, C8: 1u, Capacitor_SMD:C_0603_1608Metric, symbol Device:C
- added C22, C25, C28, C31, C34, C35, C37, C39, C41: 10n, Capacitor_SMD:C_0402_1005Metric, symbol Device:C
- added C23: 100n, Capacitor_SMD:C_0603_1608Metric, symbol Device:C
- added C42: 470n, Capacitor_SMD:C_0603_1608Metric, symbol Device:C
- added L1, L2, L3, L4, L5, L6, L7: L, Inductor_SMD:L_0603_1608Metric, symbol Device:L
- added L8: 10uH, symbol Device:L
- added R18: 150, Resistor_SMD:R_0603_1608Metric, symbol Device:R
- added U5: LM3670MFX-1.8, Package_TO_SOT_SMD:TSOT-23-5, symbol Regulator_Switching:LM3670MF
- added U6: BGT60UTR13DAiP, BGT60UTR13DAiP:BGT60UTR13DAiP, symbol BGT60UTR13DAiP:BGT60UTR13DAiP
- added U7, U8: TXU0304, Package_SO:TSSOP-14_4.4x5mm_P0.65mm, symbol TXU0304:TXU0304
- added U9: KC2016Z80.0000, Oscillator:Oscillator_SMD_Kyocera_KC2520Z-4Pin_2.5x2.0mm, symbol Oscillator:KC2520Z
- C14, C15: footprint (none) -> Capacitor_SMD:C_0603_1608Metric
- C8: value 100n -> 10n; footprint (none) -> Capacitor_SMD:C_0402_1005Metric
Connections:
- net +1V8: now also C15.1, C23.1, C26.1, C29.1, L2.1, L3.1, L4.1, L5.1, L6.1, L7.1, L8.2, U5.4 (FB), U7.14 (VCCB), U8.14 (VCCB); no longer C8.1
- net +3.3V: now also C20.1, L1.1, U5.1 (Vin), U5.3 (EN), U7.1 (VCCA), U7.8 (OE), U8.1 (VCCA), U8.8 (OE)
- net GND: now also C15.2, C20.2, C21.2, C22.2, C23.2, C24.2, C25.2, C26.2, C27.2, C28.2, C29.2, C30.2, C31.2, C32.2, C33.2, C34.2, C35.2, C36.2, C37.2, C38.2, C39.2, C40.2, C41.2, C42.2, C8.2, U5.2 (GND), U6.A1 (VSS_{RF}), U6.A2 (VSS_{D}), U6.A3 (VSS_{D}), U6.A4 (VSS_{RF}), U6.A5 (VSS_{RF}), U6.A6 (VSS_{RF}), U6.A7 (VSS_{RF}), U6.A8 (VSS_{RF}), U6.B2 (VSS_{RF}), U6.B7 (VSS_{RF}), U6.B8 (VSS_{RF}), U6.C8 (VSS_{RF}), U6.D8 (VSS_{RF}), U6.E8 (VSS_{RF}), U6.F8 (VSS_{RF}), U6.J8 (VSS_{RF}), U6.K1 (VSS_{A}), U6.K8 (VSS_{RF}), U6.L8 (VSS_{RF}), U6.M1 (VSS_{RF}), U6.M8 (VSS_{RF}), U7.7 (GND), U8.7 (GND), U9.2 (GND)
- net OSC_CLK: now also R18.2, U6.M4 (OSC_CLK)
- net RADAR_INT: now also U8.5 (A4Y)
- net RADAR_RST: now also U8.2 (A1)
- new net: R18.1, U9.3 (CLK)
- new net: L8.1, U5.5 (SW)
- new net INT_1V8: U6.C1 (IRQ), U8.10 (B4)
- new net MISO_1V8: U6.E1 (MISO), U7.10 (B4)
- new net MOSI_1V8: U6.D1 (MOSI), U7.11 (B3Y)
- new net NSS_1V8: U6.G1 (~{CS}), U7.12 (B2Y)
- new net RST_1V8: U6.F1 (RST), U8.13 (B1Y)
- new net SCK_1V8: U6.B1 (CLK), U7.13 (B1Y)
- new net SPI2_MISO: U7.5 (A4Y)
- new net SPI2_MOSI: U7.4 (A3)
- new net SPI2_NSS: U7.3 (A2)
- new net SPI2_SCK: U7.2 (A1)
- new net VDD_A: C24.1, C25.1, L2.2, U6.J1 (VDD_{A})
- new net VDD_D: C30.1, C31.1, L4.2, U6.H1 (VDD_{D})
- new net VDD_LF: C21.1, C22.1, L1.2, U6.M2 (VDD_{LF})
- new net VDD_PLL: C33.1, C34.1, L5.2, U6.M3 (VDD_{PLL})
- new net VDD_RF: C27.1, C28.1, C32.1, C35.1, C38.1, C39.1, C40.1, C41.1, L3.2, U6.G8 (VDD_{RF}), U6.H8 (VDD_{RF}), U6.M5 (VDD_{RF})
- new net VDD_VCO: C36.1, C37.1, L6.2, U6.M7 (VDD_{VCO})
- new net V_AREF: C42.1, U6.L1 (V_{AREF})
- new net V_OSC: C8.1, C8.1, L7.2, U9.1 (INH), U9.4 (VCC)
- no-connect marks 0 -> 5
Other:
- note added: "I_{max} = 10mA"
- note added: "I_{max} = 230mA"
- moved on the sheet: C14, C15, C8

Commit message: Finished routing
Parts:
- removed C14, C15 (x2): 10u, Capacitor_SMD:C_0603_1608Metric, symbol Device:C
- removed L8: 10uH, symbol Device:L
- removed U5: LM3670MFX-1.8, Package_TO_SOT_SMD:TSOT-23-5, symbol Regulator_Switching:LM3670MF
- added C12 (x2), C13: 10u, Capacitor_SMD:C_0603_1608Metric, symbol Device:C
- added C57, C58, C59, C60: 100n, Capacitor_SMD:C_0603_1608Metric, symbol Device:C
- added U3: TLV74318 SOT23-5, Package_TO_SOT_SMD:SOT-23-5, symbol Regulator_Linear:TLV70012_SOT23-5
- C25: renamed from C42; footprint Capacitor_SMD:C_0603_1608Metric -> Capacitor_SMD:C_0402_1005Metric
- R1: renamed from R18; footprint Resistor_SMD:R_0603_1608Metric -> Resistor_SMD:R_0402_1005Metric
- U2: renamed from U9; footprint Oscillator:Oscillator_SMD_Kyocera_KC2520Z-4Pin_2.5x2.0mm -> KC2016Z:KC2016Z
- renumbered C20 to C1, C23 to C11, C24 to C12, C25 to C13, C33 to C14, C34 to C15, C38 to C16, C39 to C17, C26 to C18, C27 to C19, C21 to C2, C28 to C20, C36 to C21, C37 to C22, C40 to C23, C41 to C24, C22 to C3, C29 to C4, C30 to C5, C31 to C6, C32 to C7, C35 to C8, L4 to L2, L7 to L3, L2 to L4, L3 to L6, L6 to L7, U7 to U3, U6 to U5, U8 to U6
Connections:
- net +1V8: now also U3.8 (OE), U6.8 (OE), C12.1, C12.1, C58.1, C60.1, U3.5 (OUT)
- net +3.3V: now also C13.1, C57.1, C59.1, U3.1 (IN), U3.3 (EN); no longer U3.8 (OE), U6.8 (OE)
- net GND: now also C12.2, C12.2, C13.2, C57.2, C58.2, C59.2, C60.2, U3.2 (GND)
- net INT_1V8: now also U3.10 (B4); no longer U6.10 (B4)
- net MISO_1V8: now also U6.10 (B4); no longer U3.10 (B4)
- net MOSI_1V8: now also U3.12 (B2Y); no longer U3.11 (B3Y)
- net NSS_1V8: now also U6.12 (B2Y); no longer U3.12 (B2Y)
- net RADAR_INT: now also U3.5 (A4Y); no longer U6.5 (A4Y)
- net RST_1V8: now also U6.11 (B3Y); no longer U6.13 (B1Y)
- net SCK_1V8: now also U3.11 (B3Y); no longer U3.13 (B1Y)
- net SPI2_MISO: now also U6.5 (A4Y); no longer U3.5 (A4Y)
- net SPI2_MOSI: now also U3.3 (A2); no longer U3.4 (A3)
- net SPI2_NSS: now also U6.3 (A2); no longer U3.3 (A2)
- net SPI2_SCK: now also U3.4 (A3); no longer U3.2 (A1)
- net 80mhz: now reaches R1.1, U2.3 (CLK)
- net RADAR_nRST: now reaches U6.4 (A3)
- net RADAR_RST: no longer names the net of U6.2 (A1)
Other:
- note added: "yes, this really should be 3.3V"
- moved on the sheet: C25, U5

Commit message: Add testpoints, 0ohm, led, logos
Parts:
- added R21: 0, Resistor_SMD:R_0603_1608Metric, symbol Device:R
- added TP4: MOSI, TestPoint:TestPoint_Pad_D1.0mm, symbol Connector:TestPoint
- added TP5: SCK, TestPoint:TestPoint_Pad_D1.0mm, symbol Connector:TestPoint
- added TP6: RADAR_INT, TestPoint:TestPoint_Pad_D1.0mm, symbol Connector:TestPoint
- added TP7: NSS, TestPoint:TestPoint_Pad_D1.0mm, symbol Connector:TestPoint
- added TP8: RADAR_nRST, TestPoint:TestPoint_Pad_D1.0mm, symbol Connector:TestPoint
- added TP9: MISO, TestPoint:TestPoint_Pad_D1.0mm, symbol Connector:TestPoint
Connections:
- net +3.3V: now also R21.1; no longer C1.1, C13.1, C57.1, C59.1, L1.1, U3.1 (IN), U3.1 (VCCA), U3.3 (EN), U6.1 (VCCA)
- net RADAR_INT: now also TP6.1
- net RADAR_nRST: now also TP8.1
- net SPI2_MISO: now also TP9.1
- net SPI2_MOSI: now also TP4.1
- net SPI2_NSS: now also TP7.1
- net SPI2_SCK: now also TP5.1
- new net Vradar: C1.1, C13.1, C57.1, C59.1, L1.1, R21.2, U3.1 (IN), U3.1 (VCCA), U3.3 (EN), U6.1 (VCCA)

Commit message: Final fixes, manufacturing
Parts:
- C1, C12, C13, C18, C19, C4: MANUFACTURER (none) -> Murata; MOUSER NO (none) -> 81-GRM188Z71A106KA3D; PART NO (none) -> GRM188Z71A106KA73D
- C11, C57, C58, C59, C60: MANUFACTURER (none) -> KEMET; MOUSER NO (none) -> 80-C603C104K5RAC3121; PART NO (none) -> C0603C104K5RAC3121
- C13, C15, C17, C20, C22, C24, C3, C6, C8: MANUFACTURER (none) -> Murata; MOUSER NO (none) -> 81-GRM1555C1E103GE1D; PART NO (none) -> GRM1555C1E103GE01D
- C14, C16, C2, C21, C23, C5, C7, C8: MANUFACTURER (none) -> Murata; MOUSER NO (none) -> 81-GCJ188R71E105KA1D; PART NO (none) -> GCJ188R71E105KA01D
- C25: MANUFACTURER (none) -> Murata; MOUSER NO (none) -> 81-GRT155R6YA474KE1D; PART NO (none) -> GRT155R6YA474KE01D
- L1, L2, L3, L4, L5, L6, L7: value L -> BLM15PX471SZ1D; footprint Inductor_SMD:L_0603_1608Metric -> Inductor_SMD:L_0402_1005Metric; MANUFACTURER (none) -> Murata; MOUSER NO (none) -> 81-BLM15PX471SZ1D; PART NO (none) -> BLM15PX471SZ1D
- R1: MANUFACTURER (none) -> Vishay / Dale; MOUSER NO (none) -> 71-CRCW0402-150-E3; PART NO (none) -> CRCW0402150RFKED
- R21: MANUFACTURER (none) -> Vishay / Dale; MOUSER NO (none) -> 71-CRCW06030000Z0EBC; PART NO (none) -> CRCW06030000Z0EBC
- U2: MANUFACTURER (none) -> KYOCERA AVX; MOUSER NO (none) -> 346-2016Z80.C1KX; PART NO (none) -> KC2016Z80.0000C1KX00
- U3, U6: MANUFACTURER (none) -> Texas Instruments; MOUSER NO (none) -> 595-TXU0304PWR; PART NO (none) -> TXU0304PWR
- U3: MANUFACTURER (none) -> Texas Instruments; MOUSER NO (none) -> 595-TLV74318PDBVR; PART NO (none) -> TLV74318PDBVR
