File: hardware/radartof-hardware.kicad_sch (KiCad schematic)
At the start: 0 parts

Commit message: final-ish schematic
Other:
- note added: "I_{max} = 130mA"
- note added: "I_{max} = 187.3mA"
- note added: "I_{max} ≈ 140mA"
- note removed: "TODO: - I2C pullups"
Changed lines of the file:
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@@
   (title_block
     (title "Heterogeneous radar, RGB, and ToF sensor board")
-    (date "2023-04-12")
+    (date "2023-04-17")
     (rev "0")
     (company "Center for Project-Based Learning")
     (comment 1 "Zoltán Marcsek")
   )
-  (bus_alias "USB_FS" (members "USB_FS+" "USB_FS-"))
+  (bus_alias "USB_HS" (members "USB_HS+" "USB_HS-"))
+  (bus_alias "I2C1" (members "I2C1_SDA" "I2C1_SCL"))
   (bus_alias "ETH" (members "ETH_A+" "ETH_A-" "ETH_B+" "ETH_B-" "ETH_LED1" "ETH_LED2"))
   (bus_alias "SPI2" (members "SPI2_MOSI" "SPI2_MISO" "SPI2_SCK" "SPI2_NSS"))
-  (bus_alias "I2C1" (members "I2C1_SDA" "I2C1_SCL"))
-  (bus_alias "USB_HS" (members "USB_HS+" "USB_HS-"))
   (bus_alias "I2C3" (members "I2C3_SDA" "I2C3_SCL"))
+  (bus_alias "USB_FS" (members "USB_FS+" "USB_FS-"))
   (wire (pts (xy 101.6 66.04) (xy 127 66.04))
     (stroke (width 0) (type default))
@@
     (stroke (width 0) (type default))
   )
-  (text "Pullups in tof sheet" (at 104.14 97.79 0)
+  (text_box "I_{max,total} ≈ 460mA"
+    (at 50.8 38.1 0) (size 25.4 6.35)
+    (stroke (width 0.5) (type default))
+    (fill (type none))
+    (effects (font (face "Asap") (size 2 2) (thickness 0.4) bold))
+  )
+  (text "I_{max} ≈ 140mA" (at 57.15 64.77 0)
+    (effects (font (face "Asap") (size 2 2) (thickness 0.4) bold) (justify left bottom))
+  )
+  (text "I_{max} = 130mA" (at 57.15 102.87 0)
+    (effects (font (face "Asap") (size 2 2) (thickness 0.4) bold) (justify left bottom))
+  )
+  (text "I_{max} = 187.3mA" (at 57.15 140.97 0)
+    (effects (font (face "Asap") (size 2 2) (thickness 0.4) bold) (justify left bottom))
+  )
+  (text "Pullups in tof sheet" (at 105.41 97.79 0)
     (effects (font (face "Asap") (size 1.27 1.27) (thickness 0.254) bold) (justify left bottom))
   )
-  (text "TODO:\n- I2C pullups" (at 42.9511 70.8219 0)
-    (effects (font (size 1.27 1.27)) (justify left bottom))
-  )
   (sheet (at 190.5 88.9) (size 25.4 25.4) (fields_autoplaced)

Commit message: Finished routing
Other:
- added sheet microSD socket (microsd.kicad_sch)
- sheet Portenta ports: added RADAR_nRST, {SDC}; removed RADAR_RST
- sheet Radar ports: added RADAR_nRST; removed RADAR_RST
- note added: "I_{max} = 140mA From 5V with SMPS"
- note added: "I_{max} ≈ 240mA"
- note removed: "I_{max} = 187.3mA"
- note removed: "I_{max} ≈ 140mA"
Changed lines of the file:
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@@
   (title_block
     (title "Heterogeneous radar, RGB, and ToF sensor board")
-    (date "2023-04-17")
-    (rev "0")
+    (date "2023-04-24")
+    (rev "1.2")
     (company "Center for Project-Based Learning")
     (comment 1 "Zoltán Marcsek")
   )
   (bus_alias "USB_HS" (members "USB_HS+" "USB_HS-"))
+  (bus_alias "SDC" (members "SDC_D0" "SDC_D1" "SDC_D2" "SDC_D3" "SDC_CLK" "SDC_CMD" "SDC_CD"))
+  (bus_alias "SPI2" (members "SPI2_MOSI" "SPI2_MISO" "SPI2_SCK" "SPI2_NSS"))
+  (bus_alias "USB_FS" (members "USB_FS+" "USB_FS-"))
+  (bus_alias "I2C3" (members "I2C3_SDA" "I2C3_SCL"))
   (bus_alias "I2C1" (members "I2C1_SDA" "I2C1_SCL"))
   (bus_alias "ETH" (members "ETH_A+" "ETH_A-" "ETH_B+" "ETH_B-" "ETH_LED1" "ETH_LED2"))
-  (bus_alias "SPI2" (members "SPI2_MOSI" "SPI2_MISO" "SPI2_SCK" "SPI2_NSS"))
-  (bus_alias "I2C3" (members "I2C3_SDA" "I2C3_SCL"))
-  (bus_alias "USB_FS" (members "USB_FS+" "USB_FS-"))
   (wire (pts (xy 101.6 66.04) (xy 127 66.04))
     (stroke (width 0) (type default))
@@
     (stroke (width 0) (type default))
   )
+  (bus (pts (xy 165.1 63.5) (xy 190.5 63.5))
+    (stroke (width 0) (type default))
+  )
   (wire (pts (xy 101.6 147.32) (xy 127 147.32))
     (stroke (width 0) (type default))
@@
     (stroke (width 0) (type default))
   )
-  (text_box "I_{max,total} ≈ 460mA"
-    (at 50.8 38.1 0) (size 25.4 6.35)
+  (text_box "I_{3.3V} ≈ 370mA\nI_{5V} ≈ 140mA"
+    (at 44.45 35.56 0) (size 25.4 8.89)
     (stroke (width 0.5) (type default))
     (fill (type none))
     (effects (font (face "Asap") (size 2 2) (thickness 0.4) bold))
   )
-  (text "I_{max} ≈ 140mA" (at 57.15 64.77 0)
+  (text "I_{max} ≈ 240mA" (at 50.8 64.77 0)
     (effects (font (face "Asap") (size 2 2) (thickness 0.4) bold) (justify left bottom))
   )
-  (text "I_{max} = 130mA" (at 57.15 102.87 0)
+  (text "I_{max} = 130mA" (at 50.8 102.87 0)
     (effects (font (face "Asap") (size 2 2) (thickness 0.4) bold) (justify left bottom))
   )
-  (text "I_{max} = 187.3mA" (at 57.15 140.97 0)
+  (text "I_{max} = 140mA\nFrom 5V with SMPS" (at 50.8 142.24 0)
     (effects (font (face "Asap") (size 2 2) (thickness 0.4) bold) (justify left bottom))
   )
@@
     (effects (font (face "Asap") (size 1.27 1.27) (thickness 0.254) bold) (justify left bottom))
   )
+  (sheet (at 190.5 50.8) (size 25.4 25.4) (fields_autoplaced)
+    (stroke (width 0.1524) (type solid))
+    (fill (color 0 0 0 0.0000))
+    (property "Sheetname" "microSD socket" (at 190.5 50.0884 0)
+      (effects (font (size 1.27 1.27)) (justify left bottom))
+    )
+    (property "Sheetfile" "microsd.kicad_sch" (at 190.5 76.7846 0)
+      (effects (font (size 1.27 1.27)) (justify left top))
+    )
+    (pin "{SDC}" bidirectional (at 190.5 63.5 180)
+      (effects (font (size 1.27 1.27)) (justify left))
+    )
+    (instances
+      (project "radartof-hardware"
+        (path "/03db8980-0fb1-4523-a968-8d3a1d96010b" (page "6"))
+      )
+    )
+  )
   (sheet (at 190.5 88.9) (size 25.4 25.4) (fields_autoplaced)
     (stroke (width 0.1524) (type solid))
@@
     (instances
       (project "radartof-hardware"
-        (path "/03db8980-0fb1-4523-a968-8d3a1d96010b" (page "6"))
+        (path "/03db8980-0fb1-4523-a968-8d3a1d96010b" (page "7"))
       )
     )
@@
       (effects (font (size 1.27 1.27)) (justify left))
     )
-    (pin "RADAR_RST" output (at 127 66.04 180)
-      (effects (font (size 1.27 1.27)) (justify left))
-    )
     (pin "TOF_INT" input (at 127 100.33 180)
       (effects (font (size 1.27 1.27)) (justify left))
@@
       (effects (font (size 1.27 1.27)) (justify left))
     )
+    (pin "{SDC}" bidirectional (at 165.1 63.5 0)
+      (effects (font (size 1.27 1.27)) (justify right))
+    )
+    (pin "RADAR_nRST" output (at 127 66.04 180)
+      (effects (font (size 1.27 1.27)) (justify left))
+    )
     (instances
       (project "radartof-hardware"
@@
       (effects (font (size 1.27 1.27)) (justify right))
     )
-    (pin "RADAR_RST" input (at 101.6 66.04 0)
-      (effects (font (size 1.27 1.27)) (justify right))
-    )
     (pin "{SPI2}" bidirectional (at 101.6 60.96 0)
       (effects (font (size 1.27 1.27)) (justify right))
     )
+    (pin "RADAR_nRST" input (at 101.6 66.04 0)
+      (effects (font (size 1.27 1.27)) (justify right))
+    )

Commit message: Final fixes, manufacturing
Other:
- note added: "Mouser cart for 5 boards: https://www.mouser.ch/ProjectManager/ProjectDetail.aspx?AccessID=c16bec37f3"
Changed lines of the file:
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@@
   (title_block
     (title "Heterogeneous radar, RGB, and ToF sensor board")
-    (date "2023-04-25")
-    (rev "1.3")
+    (date "2023-04-26")
+    (rev "1.4")
     (company "Center for Project-Based Learning")
     (comment 1 "Zoltán Marcsek")
   )
-  (bus_alias "SDC" (members "SDC_D0" "SDC_D1" "SDC_D2" "SDC_D3" "SDC_CLK" "SDC_CMD" "SDC_CD"))
   (bus_alias "SPI2" (members "SPI2_MOSI" "SPI2_MISO" "SPI2_SCK" "SPI2_NSS"))
+  (bus_alias "I2C1" (members "I2C1_SDA" "I2C1_SCL"))
   (bus_alias "I2C3" (members "I2C3_SDA" "I2C3_SCL"))
   (bus_alias "USB_FS" (members "USB_FS+" "USB_FS-"))
-  (bus_alias "I2C1" (members "I2C1_SDA" "I2C1_SCL"))
   (bus_alias "USB_HS" (members "USB_HS+" "USB_HS-"))
   (bus_alias "ETH" (members "ETH_A+" "ETH_A-" "ETH_B+" "ETH_B-" "ETH_LED1" "ETH_LED2"))
+  (bus_alias "SDC" (members "SDC_D0" "SDC_D1" "SDC_D2" "SDC_D3" "SDC_CLK" "SDC_CMD" "SDC_CD"))
   (wire (pts (xy 101.6 66.04) (xy 127 66.04))
     (stroke (width 0) (type default))
@@
     (effects (font (face "Asap") (size 1.27 1.27) (thickness 0.254) bold) (justify left bottom))
   )
+  (text "Mouser cart for 5 boards: https://www.mouser.ch/ProjectManager/ProjectDetail.aspx?AccessID=c16bec37f3"
+    (at 12.7 196.85 0)
+    (effects (font (face "Asap") (size 2 2)) (justify left bottom))
+  )
   (sheet (at 190.5 50.8) (size 25.4 25.4) (fields_autoplaced)
