File: hardware/tof.kicad_sch (KiCad schematic)
At the start: 11 parts, among them U2 VL53L5CXV0GC/1

Commit message: final-ish schematic
Parts:
- removed U2: VL53L5CXV0GC/1, vl53l5cx:VL53L5CXV0GC&slash_1, symbol 2023-04-03_22-58-58:VL53L5CXV0GC/1
- added U2: VL53L5CXV0GC/1, vl53l5cx:VL53L5CXV0GC&slash_1, symbol VL53L5CX:VL53L5CXV0GC/1
Connections:
- net +3.3V: now also U2.A4 (IOVDD), U2.B1 (AVDD), U2.B7 (AVDD)
- net GND: now also U2.A2 (RSVD4), U2.A6 (RSVD1), U2.A7 (RSVD2), U2.B4 (THERMAL_PAD), U2.C1 (GND), U2.C6 (RSVD3), U2.C7 (GND)
- net I2C3_SCL: now also U2.C4 (SCL)
- net I2C3_SDA: now also U2.C3 (SDA)
- net TOF_INT: now also U2.A3 (INT)
- net TOF_LPn: now also U2.A5 (LPn)
- net TOF_RST: now also U2.A1 (I2C_RST)
- net at R12.2: now also U2.C2 (RSVD6)

Commit message: Finished routing
Parts:
- added C55: 100n, Capacitor_SMD:C_0402_1005Metric, symbol Device:C
- C29: renamed from C3; footprint Capacitor_SMD:C_0603_1608Metric -> Capacitor_SMD:C_0402_1005Metric
- C30: renamed from C4; footprint Capacitor_SMD:C_0603_1608Metric -> Capacitor_SMD:C_0402_1005Metric
- C31: renamed from C5; footprint Capacitor_SMD:C_0603_1608Metric -> Capacitor_SMD:C_0402_1005Metric
- renumbered C2 to C28, R11 to R2, R10 to R3, R9 to R4, R8 to R5, R12 to R6, U2 to U7
Connections:
- net +3.3V: now also C55.1
- net GND: now also C55.2
- net RSVD6: now reaches R6.2, U7.C2 (RSVD6)
Other:
- note added: "C55 is bypass for reference change"

Commit message: Add testpoints, 0ohm, led, logos
Parts:
- added R21: 0, Resistor_SMD:R_0603_1608Metric, symbol Device:R
- added TP4: SDA3, TestPoint:TestPoint_Pad_D1.0mm, symbol Connector:TestPoint
- added TP4: TOF_LPn, TestPoint:TestPoint_Pad_D1.0mm, symbol Connector:TestPoint
- added TP4: TOF_INT, TestPoint:TestPoint_Pad_D1.0mm, symbol Connector:TestPoint
- added TP4: TOF_RST, TestPoint:TestPoint_Pad_D1.0mm, symbol Connector:TestPoint
- added TP4: SCL3, TestPoint:TestPoint_Pad_D1.0mm, symbol Connector:TestPoint
Connections:
- net +3.3V: now also R21.1; no longer C28.1, C29.1, C30.1, C31.1, R6.1, U7.A4 (IOVDD), U7.B1 (AVDD), U7.B7 (AVDD)
- net I2C3_SCL: now also TP4.1
- net I2C3_SDA: now also TP4.1
- net TOF_INT: now also TP4.1
- net TOF_LPn: now also TP4.1
- net TOF_RST: now also TP4.1
- new net VTOF: C28.1, C29.1, C30.1, C31.1, R21.2, R6.1, U7.A4 (IOVDD), U7.B1 (AVDD), U7.B7 (AVDD)

Commit message: Final fixes, manufacturing
Parts:
- C28: MANUFACTURER (none) -> Murata; MOUSER NO (none) -> 81-GRT188C71C475KE13; PART NO (none) -> GRT188C71C475KE13D
- C29, C30, C31, C55: MANUFACTURER (none) -> Murata; MOUSER NO (none) -> 81-GRM155R71H104KE4D; PART NO (none) -> GRM155R71H104KE14D
- R2, R3: MANUFACTURER (none) -> Vishay / Dale; MOUSER NO (none) -> 71-CRCW06032K20FKEAC; PART NO (none) -> CRCW06032K20FKEAC
- R21: MANUFACTURER (none) -> Vishay / Dale; MOUSER NO (none) -> 71-CRCW06030000Z0EBC; PART NO (none) -> CRCW06030000Z0EBC
- R4, R5, R6, R7: MANUFACTURER (none) -> Vishay / Dale; MOUSER NO (none) -> 71-CRCW060347K0FKEAC; PART NO (none) -> CRCW060347K0FKEAC
- U7: MANUFACTURER (none) -> STMicroelectronics; MOUSER NO (none) -> 511-VL53L5CXV0GC/1; PART NO (none) -> VL53L5CXV0GC/1

Commit message: Manufacturing
Changed lines of the file:
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@@
     )
     (property "Datasheet" "https://www.st.com/resource/en/datasheet/vl53l5cx.pdf" (at 116.84 77.47 0)
-      (effects (font (size 1.524 1.524)))
+      (effects (font (size 1.524 1.524)) hide)
     )
     (property "MOUSER NO" "511-VL53L5CXV0GC/1" (at 139.7 101.6 0)
